File: Fuzz/Fuzz.kicad_pcb (KiCad board)
At the start: 2 copper layers, 33.7 x 38.4 mm, 21 parts, among them J1 AudioJack3, J2 AudioJack2, Q1 BC109, Q2 BC109, SW1 SW_SPST, SW2 SW_SPST, SW3 SW_SPST

Commit message: updated values
Parts:
- removed REF** (x2): MountingHole_3.2mm_M3, MountingHole:MountingHole_3.2mm_M3
- C1: value CP1 -> 2.2uf
- C2: value C -> 0.01uf
- C3: value CP1 -> 22uf
- Pot1: value R_POT -> 1K
- Pot2: value R_POT -> 500K
- R1: value R -> 33K
- R2, R5: value R -> 100K
- R3: value R -> 330
- R4: value R -> 8.2K

Commit message: Added gerber files
Other:
- board text added: "+"
