File: MuffPiSMT/MuffPiSMT.sch (KiCad schematic (older format))
At the start: 52 parts, among them J1 AudioJack3, J2 AudioJack2, Q1 2N3904, Q2 2N3904, Q3 2N3904, Q4 2N3904

Commit message: Minor Changes
Parts:
- R1: LCSC (none) -> C4216
- R2, R23, R8: LCSC (none) -> C25803
Changed lines of the file:
@@
 F 2 "Resistor_SMD:R_0603_1608Metric" V 2630 4100 50  0001 C CNN
 F 3 "~" H 2700 4100 50  0001 C CNN
+F 4 "C4216" V 2700 4100 50  0001 C CNN "LCSC"
 	1    2700 4100
 	0    1    1    0
@@
 F 2 "Resistor_SMD:R_0603_1608Metric" V 3080 4550 50  0001 C CNN
 F 3 "~" H 3150 4550 50  0001 C CNN
+F 4 "C25803" H 3150 4550 50  0001 C CNN "LCSC"
 	1    3150 4550
 	-1   0    0    1
@@
 F 2 "Resistor_SMD:R_0603_1608Metric" V 5030 4550 50  0001 C CNN
 F 3 "~" H 5100 4550 50  0001 C CNN
+F 4 "C25803" H 5100 4550 50  0001 C CNN "LCSC"
 	1    5100 4550
 	1    0    0    -1
@@
 F 2 "Resistor_SMD:R_0603_1608Metric" V 2530 1750 50  0001 C CNN
 F 3 "~" H 2600 1750 50  0001 C CNN
+F 4 "C25803" V 2600 1750 50  0001 C CNN "LCSC"
 	1    2600 1750
 	0    -1   -1   0

Commit message: minor changes
Parts:
- J1: symbol MuffPi3PDT-rescue:AudioJack3-Connector-MuffPi-rescue -> Connector:AudioJack3
- J2: symbol MuffPi3PDT-rescue:AudioJack2-Connector-MuffPi-rescue -> Connector:AudioJack2
Connections:
- net GND: now also J1.S, J2.S; no longer J1.1, J2.2
- net at S1.P$7 (O): now also J2.T; no longer J2.1
- net at BT1.2 (-): now also J1.R; no longer J1.2
- net at S1.P$5 (P): now also J1.T; no longer J1.3
Changed lines of the file:
@@
 $EndDescr
 $Comp
-L MuffPi3PDT-rescue:AudioJack2-Connector-MuffPi-rescue J2
+L Connector:AudioJack2 J2
 U 1 1 5F95CCEC
 P 10100 4100
@@
 $EndComp
 $Comp
-L MuffPi3PDT-rescue:AudioJack3-Connector-MuffPi-rescue J1
+L Connector:AudioJack3 J1
 U 1 1 5F95E152
 P 1500 4000

Commit message: Finalized SMT CSV's. Placed order for PCBs based on this version
Parts:
- S1: symbol MuffPi:SWITCH-3PDT-PTH-STOMP -> MuffPiSMT-rescue:SWITCH-3PDT-PTH-STOMP-MuffPi
Changed lines of the file:
@@
 $EndComp
 $Comp
-L MuffPi:SWITCH-3PDT-PTH-STOMP S1
+L MuffPiSMT-rescue:SWITCH-3PDT-PTH-STOMP-MuffPi S1
 U 1 1 5F98BD88
 P 2550 2150
@@
 $EndComp
 $Comp
-L MuffPi:SWITCH-3PDT-PTH-STOMP S1
+L MuffPiSMT-rescue:SWITCH-3PDT-PTH-STOMP-MuffPi S1
 U 2 1 5F98DCFB
 P 2150 4200
@@
 $EndComp
 $Comp
-L MuffPi:SWITCH-3PDT-PTH-STOMP S1
+L MuffPiSMT-rescue:SWITCH-3PDT-PTH-STOMP-MuffPi S1
 U 3 1 5F98F300
 P 9600 4200
