File: ConsolePedalPhase/ConsolePedalPhase.sch (KiCad schematic (older format))
At the start: 53 parts, among them J1 Conn_02x25_Counter_Clockwise, SW1 SW_DPDT_x2, U1 TL072, U2 TL074, U3 CD4046BE

Commit message: Assigned some footprints
Parts:
- C10, C11, C5: footprint (none) -> Capacitor_SMD:C_0603_1608Metric
- D3: footprint Diode_THT:D_DO-41_SOD81_P10.16mm_Horizontal -> Diode_SMD:D_SOD-123
- RV1: footprint (none) -> Resistor_SMD:R_0603_1608Metric
- RV2: footprint (none) -> Connector_PinSocket_2.54mm:PinSocket_1x03_P2.54mm_Vertical
- U1: footprint (none) -> Package_SO:SOIC-8_3.9x4.9mm_P1.27mm
- U2: footprint (none) -> Package_SO:SOIC-14_3.9x8.7mm_P1.27mm
- U3: footprint DIP794W45P254L1969H508Q16 -> CD4046BE:DIP794W45P254L1969H508Q16
Changed lines of the file:
@@
 F 0 "U1" H 1850 933 50  0000 C CNN
 F 1 "TL072" H 1850 1024 50  0000 C CNN
-F 2 "" H 1850 1300 50  0001 C CNN
+F 2 "Package_SO:SOIC-8_3.9x4.9mm_P1.27mm" H 1850 1300 50  0001 C CNN
 F 3 "http://www.ti.com/lit/ds/symlink/tl071.pdf" H 1850 1300 50  0001 C CNN
 	1    1850 1300
@@
 F 0 "U1" H 5800 3833 50  0000 C CNN
 F 1 "TL072" H 5800 3924 50  0000 C CNN
-F 2 "" H 5800 4200 50  0001 C CNN
+F 2 "Package_SO:SOIC-8_3.9x4.9mm_P1.27mm" H 5800 4200 50  0001 C CNN
 F 3 "http://www.ti.com/lit/ds/symlink/tl071.pdf" H 5800 4200 50  0001 C CNN
 	2    5800 4200
@@
 F 0 "U1" H 2708 6396 50  0000 L CNN
 F 1 "TL072" H 2708 6305 50  0000 L CNN
-F 2 "" H 2750 6350 50  0001 C CNN
+F 2 "Package_SO:SOIC-8_3.9x4.9mm_P1.27mm" H 2750 6350 50  0001 C CNN
 F 3 "http://www.ti.com/lit/ds/symlink/tl071.pdf" H 2750 6350 50  0001 C CNN
 	3    2750 6350
@@
 F 0 "U2" H 3150 933 50  0000 C CNN
 F 1 "TL074" H 3150 1024 50  0000 C CNN
-F 2 "" H 3100 1400 50  0001 C CNN
+F 2 "Package_SO:SOIC-14_3.9x8.7mm_P1.27mm" H 3100 1400 50  0001 C CNN
 F 3 "http://www.ti.com/lit/ds/symlink/tl071.pdf" H 3200 1500 50  0001 C CNN
 	1    3150 1300
@@
 F 0 "U2" H 5250 833 50  0000 C CNN
 F 1 "TL074" H 5250 924 50  0000 C CNN
-F 2 "" H 5200 1300 50  0001 C CNN
+F 2 "Package_SO:SOIC-14_3.9x8.7mm_P1.27mm" H 5200 1300 50  0001 C CNN
 F 3 "http://www.ti.com/lit/ds/symlink/tl071.pdf" H 5300 1400 50  0001 C CNN
 	2    5250 1200
@@
 F 0 "U2" H 6400 6133 50  0000 C CNN
 F 1 "TL074" H 6400 6224 50  0000 C CNN
-F 2 "" H 6350 6600 50  0001 C CNN
+F 2 "Package_SO:SOIC-14_3.9x8.7mm_P1.27mm" H 6350 6600 50  0001 C CNN
 F 3 "http://www.ti.com/lit/ds/symlink/tl071.pdf" H 6450 6700 50  0001 C CNN
 	3    6400 6500
@@
 F 0 "U2" H 6250 1467 50  0000 C CNN
 F 1 "TL074" H 6250 1376 50  0000 C CNN
-F 2 "" H 6200 1200 50  0001 C CNN
+F 2 "Package_SO:SOIC-14_3.9x8.7mm_P1.27mm" H 6200 1200 50  0001 C CNN
 F 3 "http://www.ti.com/lit/ds/symlink/tl071.pdf" H 6300 1300 50  0001 C CNN
 	4    6250 1100
@@
 F 0 "U2" H 3108 6396 50  0000 L CNN
 F 1 "TL074" H 3108 6305 50  0000 L CNN
-F 2 "" H 3100 6450 50  0001 C CNN
+F 2 "Package_SO:SOIC-14_3.9x8.7mm_P1.27mm" H 3100 6450 50  0001 C CNN
 F 3 "http://www.ti.com/lit/ds/symlink/tl071.pdf" H 3200 6550 50  0001 C CNN
 	5    3150 6350
@@
 F 0 "U3" H 9200 4020 50  0000 C CNN
 F 1 "CD4046BE" H 9200 3929 50  0000 C CNN
-F 2 "DIP794W45P254L1969H508Q16" H 9200 2950 50  0001 L BNN
+F 2 "CD4046BE:DIP794W45P254L1969H508Q16" H 9200 2950 50  0001 L BNN
 F 3 "" H 9200 2950 50  0001 L BNN
 	1    9200 2950
@@
 F 0 "RV1" H 1931 3096 50  0000 R CNN
 F 1 "20K" H 1931 3005 50  0000 R CNN
-F 2 "" H 2000 3050 50  0001 C CNN
+F 2 "Resistor_SMD:R_0603_1608Metric" H 2000 3050 50  0001 C CNN
 F 3 "~" H 2000 3050 50  0001 C CNN
 	1    2000 3050
@@
 F 0 "C11" V 4605 3600 50  0000 C CNN
 F 1 "10uF" V 4514 3600 50  0000 C CNN
-F 2 "" H 4388 3450 50  0001 C CNN
+F 2 "Capacitor_SMD:C_0603_1608Metric" H 4388 3450 50  0001 C CNN
 F 3 "~" H 4350 3600 50  0001 C CNN
 	1    4350 3600
@@
 F 0 "RV2" V 4735 3600 50  0000 C CNN
 F 1 "C100K" V 4644 3600 50  0000 C CNN
-F 2 "" H 4850 3600 50  0001 C CNN
+F 2 "Connector_PinSocket_2.54mm:PinSocket_1x03_P2.54mm_Vertical" H 4850 3600 50  0001 C CNN
 F 3 "~" H 4850 3600 50  0001 C CNN
 	1    4850 3600
@@
 F 0 "D3" V 3504 6430 50  0000 L CNN
 F 1 "1N5817" V 3595 6430 50  0000 L CNN
-F 2 "Diode_THT:D_DO-41_SOD81_P10.16mm_Horizontal" H 3550 6175 50  0001 C CNN
+F 2 "Diode_SMD:D_SOD-123" H 3550 6175 50  0001 C CNN
 F 3 "http://www.vishay.com/docs/88525/1n5817.pdf" H 3550 6350 50  0001 C CNN
 	1    3550 6350
@@
 F 0 "C5" H 4150 6350 50  0000 L CNN
 F 1 "100uF" H 4100 6250 50  0000 L CNN
-F 2 "" H 4088 6200 50  0001 C CNN
+F 2 "Capacitor_SMD:C_0603_1608Metric" H 4088 6200 50  0001 C CNN
 F 3 "~" H 4050 6350 50  0001 C CNN
 	1    4050 6350
@@
 F 0 "C10" H 5468 6546 50  0000 L CNN
 F 1 "100uF" H 5468 6455 50  0000 L CNN
-F 2 "" H 5388 6350 50  0001 C CNN
+F 2 "Capacitor_SMD:C_0603_1608Metric" H 5388 6350 50  0001 C CNN
 F 3 "~" H 5350 6500 50  0001 C CNN
 	1    5350 6500

Commit message: Added DPDT switch footprint
Parts:
- added C19: 100nF, Capacitor_SMD:C_0603_1608Metric, symbol Device:C
- added R25: 10K, Resistor_SMD:R_0603_1608Metric, symbol Device:R
- added TP1: CV_IN, Connector_PinSocket_2.54mm:PinSocket_1x01_P2.54mm_Vertical, symbol Connector:TestPoint
- RV1: footprint Resistor_SMD:R_0603_1608Metric -> Connector_PinSocket_2.54mm:PinSocket_1x03_P2.54mm_Vertical
- RV3: footprint (none) -> Connector_PinSocket_2.54mm:PinSocket_1x03_P2.54mm_Vertical
- SW1: footprint (none) -> libraries:DPDTSwitch
Connections:
- wire segments 141 -> 150
Changed lines of the file:
@@
 F 0 "SW1" H 2850 3300 50  0000 C CNN
 F 1 "SW_DPDT_x2" H 2800 3400 50  0000 C CNN
-F 2 "" H 2900 3150 50  0001 C CNN
+F 2 "libraries:DPDTSwitch" H 2900 3150 50  0001 C CNN
 F 3 "~" H 2900 3150 50  0001 C CNN
 	2    2900 3150
@@
 F 0 "SW1" H 1000 2425 50  0000 C CNN
 F 1 "SW_DPDT_x2" H 1000 2516 50  0000 C CNN
-F 2 "" H 1000 2750 50  0001 C CNN
+F 2 "libraries:DPDTSwitch" H 1000 2750 50  0001 C CNN
 F 3 "~" H 1000 2750 50  0001 C CNN
 	1    1000 2750
@@
 F 0 "RV3" H 6580 1754 50  0000 R CNN
 F 1 "1M" H 6580 1845 50  0000 R CNN
-F 2 "" H 6650 1800 50  0001 C CNN
+F 2 "Connector_PinSocket_2.54mm:PinSocket_1x03_P2.54mm_Vertical" H 6650 1800 50  0001 C CNN
 F 3 "~" H 6650 1800 50  0001 C CNN
 	1    6650 1800
@@
 F 0 "RV1" H 1931 3096 50  0000 R CNN
 F 1 "20K" H 1931 3005 50  0000 R CNN
-F 2 "Resistor_SMD:R_0603_1608Metric" H 2000 3050 50  0001 C CNN
+F 2 "Connector_PinSocket_2.54mm:PinSocket_1x03_P2.54mm_Vertical" H 2000 3050 50  0001 C CNN
 F 3 "~" H 2000 3050 50  0001 C CNN
 	1    2000 3050
@@
 Wire Wire Line
 	6700 5900 6700 6500
+Text GLabel 8100 4450 0    50   Input ~ 0
+VCO_IN
+Text GLabel 8100 4650 0    50   Input ~ 0
+PH_COMP2_OUT
+$Comp
+L Device:R R25
+U 1 1 5FAB2387
+P 8450 4550
+F 0 "R25" V 8650 4550 50  0000 L CNN
+F 1 "10K" V 8550 4500 50  0000 L CNN
+F 2 "Resistor_SMD:R_0603_1608Metric" V 8380 4550 50  0001 C CNN
+F 3 "~" H 8450 4550 50  0001 C CNN
+	1    8450 4550
+	0    1    1    0
+$EndComp
+Wire Wire Line
+	8300 4550 8200 4550
+Wire Wire Line
+	8200 4550 8200 4450
+Wire Wire Line
+	8200 4450 8100 4450
+Wire Wire Line
+	8100 4650 8200 4650
+Wire Wire Line
+	8200 4650 8200 4550
+Connection ~ 8200 4550
+$Comp
+L Device:C C19
+U 1 1 5FABFDD0
+P 8950 4550
+F 0 "C19" V 9000 4600 50  0000 L CNN
+F 1 "100nF" V 9100 4450 50  0000 L CNN
+F 2 "Capacitor_SMD:C_0603_1608Metric" H 8988 4400 50  0001 C CNN
+F 3 "~" H 8950 4550 50  0001 C CNN
+	1    8950 4550
+	0    1    1    0
+$EndComp
+Wire Wire Line
+	8800 4550 8700 4550
+$Comp
+L power:GND #PWR0126
+U 1 1 5FAD2C29
+P 9350 4550
+F 0 "#PWR0126" H 9350 4300 50  0001 C CNN
+F 1 "GND" H 9355 4377 50  0000 C CNN
+F 2 "" H 9350 4550 50  0001 C CNN
+F 3 "" H 9350 4550 50  0001 C CNN
+	1    9350 4550
+	1    0    0    -1
+$EndComp
+Wire Wire Line
+	9350 4550 9100 4550
+Wire Wire Line
+	8700 4900 8700 4550
+Connection ~ 8700 4550
+Wire Wire Line
+	8700 4550 8600 4550
+$Comp
+L Connector:TestPoint TP1
+U 1 1 5FAE1440
+P 8700 4900
+F 0 "TP1" H 8642 4926 50  0000 R CNN
+F 1 "CV_IN" H 8650 5000 50  0000 R CNN
+F 2 "Connector_PinSocket_2.54mm:PinSocket_1x01_P2.54mm_Vertical" H 8900 4900 50  0001 C CNN
+F 3 "~" H 8900 4900 50  0001 C CNN
+	1    8700 4900
+	-1   0    0    1
+$EndComp
 $EndSCHEMATC

Commit message: minor changes
Parts:
- removed TP1: CV_IN, Connector_PinSocket_2.54mm:PinSocket_1x01_P2.54mm_Vertical, symbol Connector:TestPoint
- added J2: AudioJack2, Connector_Audio:Jack_3.5mm_CUI_SJ1-3535NG_Horizontal, symbol Connector:AudioJack2
- RV1, RV2, RV3: footprint Connector_PinSocket_2.54mm:PinSocket_1x03_P2.54mm_Vertical -> Potentiometer_THT:Potentiometer_Alps_RK09L_Single_Vertical
- U3: footprint CD4046BE:DIP794W45P254L1969H508Q16 -> Package_SO:SOP-16_3.9x9.9mm_P1.27mm
Connections:
- wire segments 150 -> 153
Changed lines of the file:
@@
 F 0 "U3" H 9200 4020 50  0000 C CNN
 F 1 "CD4046BE" H 9200 3929 50  0000 C CNN
-F 2 "CD4046BE:DIP794W45P254L1969H508Q16" H 9200 2950 50  0001 L BNN
+F 2 "Package_SO:SOP-16_3.9x9.9mm_P1.27mm" H 9200 2950 50  0001 L BNN
 F 3 "" H 9200 2950 50  0001 L BNN
 	1    9200 2950
@@
 F 0 "RV3" H 6580 1754 50  0000 R CNN
 F 1 "1M" H 6580 1845 50  0000 R CNN
-F 2 "Connector_PinSocket_2.54mm:PinSocket_1x03_P2.54mm_Vertical" H 6650 1800 50  0001 C CNN
+F 2 "Potentiometer_THT:Potentiometer_Alps_RK09L_Single_Vertical" H 6650 1800 50  0001 C CNN
 F 3 "~" H 6650 1800 50  0001 C CNN
 	1    6650 1800
@@
 F 0 "RV1" H 1931 3096 50  0000 R CNN
 F 1 "20K" H 1931 3005 50  0000 R CNN
-F 2 "Connector_PinSocket_2.54mm:PinSocket_1x03_P2.54mm_Vertical" H 2000 3050 50  0001 C CNN
+F 2 "Potentiometer_THT:Potentiometer_Alps_RK09L_Single_Vertical" H 2000 3050 50  0001 C CNN
 F 3 "~" H 2000 3050 50  0001 C CNN
 	1    2000 3050
@@
 F 0 "RV2" V 4735 3600 50  0000 C CNN
 F 1 "C100K" V 4644 3600 50  0000 C CNN
-F 2 "Connector_PinSocket_2.54mm:PinSocket_1x03_P2.54mm_Vertical" H 4850 3600 50  0001 C CNN
+F 2 "Potentiometer_THT:Potentiometer_Alps_RK09L_Single_Vertical" H 4850 3600 50  0001 C CNN
 F 3 "~" H 4850 3600 50  0001 C CNN
 	1    4850 3600
@@
 Wire Wire Line
 	8700 4550 8600 4550
-$Comp
-L Connector:TestPoint TP1
-U 1 1 5FAE1440
-P 8700 4900
-F 0 "TP1" H 8642 4926 50  0000 R CNN
-F 1 "CV_IN" H 8650 5000 50  0000 R CNN
-F 2 "Connector_PinSocket_2.54mm:PinSocket_1x01_P2.54mm_Vertical" H 8900 4900 50  0001 C CNN
-F 3 "~" H 8900 4900 50  0001 C CNN
-	1    8700 4900
-	-1   0    0    1
+Wire Wire Line
+	9350 4550 9650 4550
+Wire Wire Line
+	9650 4550 9650 4800
+Connection ~ 9350 4550
+Wire Wire Line
+	9650 4900 8700 4900
+$Comp
+L Connector:AudioJack2 J2
+U 1 1 5FB8FB4E
+P 9850 4900
+F 0 "J2" H 9670 4975 50  0000 R CNN
+F 1 "AudioJack2" H 9670 4884 50  0000 R CNN
+F 2 "Connector_Audio:Jack_3.5mm_CUI_SJ1-3535NG_Horizontal" H 9850 4900 50  0001 C CNN
+F 3 "~" H 9850 4900 50  0001 C CNN
+	1    9850 4900
+	-1   0    0    -1
 $EndComp
 $EndSCHEMATC

Commit message: Fixed issues with library loading
Parts:
- added H1, H2: MountingHole_Pad, MountingHole:MountingHole_2.5mm_Pad, symbol Mechanical:MountingHole_Pad
- U3: symbol CD4046BE:CD4046BE -> ConsolePedalPhase-rescue:CD4046BE-CD4046BE-ConsolePedalPhase-rescue
Connections:
- net GND: now also H1.1, H2.1
Changed lines of the file:
@@
 $EndComp
 $Comp
-L CD4046BE:CD4046BE U3
+L ConsolePedalPhase-rescue:CD4046BE-CD4046BE-ConsolePedalPhase-rescue U3
 U 1 1 5FB99F22
 P 9200 2950
@@
 	-1   0    0    -1
 $EndComp
+$Comp
+L Mechanical:MountingHole_Pad H2
+U 1 1 5FACC9BD
+P 8450 5600
+F 0 "H2" H 8400 5900 50  0000 L CNN
+F 1 "MountingHole_Pad" H 8150 5800 50  0000 L CNN
+F 2 "MountingHole:MountingHole_2.5mm_Pad" H 8450 5600 50  0001 C CNN
+F 3 "~" H 8450 5600 50  0001 C CNN
+	1    8450 5600
+	1    0    0    -1
+$EndComp
+$Comp
+L Mechanical:MountingHole_Pad H1
+U 1 1 5FACCD34
+P 7600 5600
+F 0 "H1" H 7550 5900 50  0000 L CNN
+F 1 "MountingHole_Pad" H 7250 5800 50  0000 L CNN
+F 2 "MountingHole:MountingHole_2.5mm_Pad" H 7600 5600 50  0001 C CNN
+F 3 "~" H 7600 5600 50  0001 C CNN
+	1    7600 5600
+	1    0    0    -1
+$EndComp
+$Comp
+L power:GND #PWR0127
+U 1 1 5FAE1AA5
+P 8450 5700
+F 0 "#PWR0127" H 8450 5450 50  0001 C CNN
+F 1 "GND" H 8455 5527 50  0000 C CNN
+F 2 "" H 8450 5700 50  0001 C CNN
+F 3 "" H 8450 5700 50  0001 C CNN
+	1    8450 5700
+	1    0    0    -1
+$EndComp
+$Comp
+L power:GND #PWR0128
+U 1 1 5FAE1DDD
+P 7600 5700
+F 0 "#PWR0128" H 7600 5450 50  0001 C CNN
+F 1 "GND" H 7605 5527 50  0000 C CNN
+F 2 "" H 7600 5700 50  0001 C CNN
+F 3 "" H 7600 5700 50  0001 C CNN
+	1    7600 5700
+	1    0    0    -1
+$EndComp
 $EndSCHEMATC

Commit message: Fixed footprints and moved around polarized capacitors. Ready for SMT part selection
Parts:
- C10, C5: footprint Capacitor_SMD:C_0603_1608Metric -> Capacitor_SMD:CP_Elec_6.3x5.3
- C11: footprint Capacitor_SMD:C_0603_1608Metric -> Capacitor_SMD:CP_Elec_4x5.3
Changed lines of the file:
@@
 F 0 "C11" V 4605 3600 50  0000 C CNN
 F 1 "10uF" V 4514 3600 50  0000 C CNN
-F 2 "Capacitor_SMD:C_0603_1608Metric" H 4388 3450 50  0001 C CNN
+F 2 "Capacitor_SMD:CP_Elec_4x5.3" H 4388 3450 50  0001 C CNN
 F 3 "~" H 4350 3600 50  0001 C CNN
 	1    4350 3600
@@
 F 0 "C5" H 4150 6350 50  0000 L CNN
 F 1 "100uF" H 4100 6250 50  0000 L CNN
-F 2 "Capacitor_SMD:C_0603_1608Metric" H 4088 6200 50  0001 C CNN
+F 2 "Capacitor_SMD:CP_Elec_6.3x5.3" H 4088 6200 50  0001 C CNN
 F 3 "~" H 4050 6350 50  0001 C CNN
 	1    4050 6350
@@
 F 0 "C10" H 5468 6546 50  0000 L CNN
 F 1 "100uF" H 5468 6455 50  0000 L CNN
-F 2 "Capacitor_SMD:C_0603_1608Metric" H 5388 6350 50  0001 C CNN
+F 2 "Capacitor_SMD:CP_Elec_6.3x5.3" H 5388 6350 50  0001 C CNN
 F 3 "~" H 5350 6500 50  0001 C CNN
 	1    5350 6500
