File: ConsolePedalScreamer/ConsolePedalScreamer.sch (KiCad schematic (older format))
At the start: 29 parts, among them J1 Conn_02x25_Counter_Clockwise, Q1 2N3904, Q2 2N3904

Commit message: Finalized schematic
Parts:
- removed C1: 2.2uF, Capacitor_THT:CP_Axial_L11.0mm_D5.0mm_P18.00mm_Horizontal, symbol Device:CP
- removed C2: 0.01uF, Capacitor_THT:C_Disc_D10.5mm_W5.0mm_P7.50mm, symbol Device:C
- removed Q1, Q2: 2N3904, Package_TO_SOT_THT:TO-92_Inline, symbol Transistor_BJT:2N3904
- removed R1: 33K, Resistor_THT:R_Axial_DIN0207_L6.3mm_D2.5mm_P10.16mm_Horizontal, symbol Device:R
- removed R2: 330, Resistor_THT:R_Axial_DIN0207_L6.3mm_D2.5mm_P10.16mm_Horizontal, symbol Device:R
- removed R4: 100K, Resistor_THT:R_Axial_DIN0207_L6.3mm_D2.5mm_P10.16mm_Horizontal, symbol Device:R
- removed RV1: 1K, Potentiometer_THT:Potentiometer_Bourns_PTV09A-1_Single_Vertical, symbol Device:R_POT
- added C10, C5, C8, C9: 100nF, symbol Device:C
- added C6: 1.5nF, symbol Device:C
- added C7: 150pF, symbol Device:C
- added D3, D4: 1N4148, Diode_THT:D_DO-35_SOD27_P7.62mm_Horizontal, symbol Diode:1N4148
- added R10: 10K, Resistor_THT:R_Axial_DIN0207_L6.3mm_D2.5mm_P10.16mm_Horizontal, symbol Device:R
- added R11, R13, R9: 100K, Resistor_THT:R_Axial_DIN0207_L6.3mm_D2.5mm_P10.16mm_Horizontal, symbol Device:R
- added R12, R14: 220K, Resistor_THT:R_Axial_DIN0207_L6.3mm_D2.5mm_P10.16mm_Horizontal, symbol Device:R
- C1, C2, C4: renamed from C?; footprint Capacitor_THT:C_Disc_D10.5mm_W5.0mm_P7.50mm -> (none)
- C3: value 22uF -> 100uF; footprint Capacitor_THT:CP_Axial_L11.0mm_D6.0mm_P18.00mm_Horizontal -> (none)
- RV2: value 500K -> 500KL
- RV3: value 10K -> 100KL; footprint Potentiometer_THT:Potentiometer_Bourns_3386F_Vertical -> Potentiometer_THT:Potentiometer_Bourns_PTV09A-1_Single_Vertical
- U1: renamed from U?; footprint DIP794W45P254L1969H508Q16 -> CD4049UBE:DIP794W45P254L1969H508Q16
- gave numbers to parts that had none: 8
Connections:
- net pin1 is gone; now on net +9V: U1.1 (VCC)
- net pin5 is gone; now on net GND: U1.5 (B)
- net pin8 is gone; now on net GND: U1.8 (VSS)
- net +9V: now also C3.1
- net GND: now also RV3.1, C6.1; no longer RV2.3
- net Output: now also RV3.2; no longer RV2.2
- net pin11: now also D3.1 (K), D4.2 (A)
- net pin12: now also R8.2, C5.2, D3.2 (A), D4.1 (K)
- net pin14: now also RV2.1, RV2.2, C7.2
- net pin15: now also C7.1, C9.2, R11.2
- net pin2: now also C10.2, R14.2
- net pin3: now also R12.2, R13.2, R14.1
- net pin6: now also C2.2, R4.2, C8.2
- net at RV3.3: now also C10.1
- net pin4: no longer names the net of U1.4 (H_=_~B)
- new net: C5.1, R9.1
- new net: C6.2, R10.1, R11.1, R9.2
- new net: R10.2, RV2.3
- new net: C9.1, R13.1
- new net: C8.1, R12.1
Other:
- moved on the sheet: C1, C2, C4, D1, D2, H1, H2, J1, R1, R2, R3, R4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

Commit message: Finalized and plotted new board
Parts:
- C1, C10, C2, C4, C5, C6, C8, C9: footprint (none) -> libraries:C_Flat_L7.2_H6.5
- C3: footprint (none) -> Capacitor_THT:CP_Axial_L10.0mm_D6.0mm_P15.00mm_Horizontal
- C7: footprint (none) -> Capacitor_THT:C_Axial_L5.1mm_D3.1mm_P10.00mm_Horizontal
Connections:
- net GND: now also RV3.3; no longer RV3.1
- net pin14: now also RV2.3; no longer RV2.1
- net at RV1.1: now also R7.1; no longer R6.2
- net at RV1.3: now also R6.2; no longer R7.1
- net at R10.2: now also RV2.1; no longer RV2.3
- net at C10.1: now also RV3.1; no longer RV3.3
Changed lines of the file:
@@
 F 0 "C1" V 1448 3300 50  0000 C CNN
 F 1 "10nF" V 1539 3300 50  0000 C CNN
-F 2 "" H 1738 3150 50  0001 C CNN
+F 2 "libraries:C_Flat_L7.2_H6.5" H 1738 3150 50  0001 C CNN
 F 3 "~" H 1700 3300 50  0001 C CNN
 	1    1700 3300
@@
 	0    -1   -1   0
 $EndComp
-Text GLabel 6550 6500 2    50   Input ~ 0
-pin1
-Text GLabel 6550 6700 2    50   Input ~ 0
-pin2
-Text GLabel 6550 6900 2    50   Input ~ 0
-pin6
-Text GLabel 6550 7000 2    50   Input ~ 0
-pin10
-Text GLabel 6550 7100 2    50   Input ~ 0
-pin12
-Text GLabel 6550 7200 2    50   Input ~ 0
-pin15
-Text GLabel 6550 7400 2    50   Input ~ 0
-pin8
-Text GLabel 5150 6700 0    50   Input ~ 0
-pin3
-Text GLabel 5150 6800 0    50   Input ~ 0
-pin5
-Text GLabel 5150 6900 0    50   Input ~ 0
-pin7
-Text GLabel 5150 7000 0    50   Input ~ 0
-pin9
-Text GLabel 5150 7100 0    50   Input ~ 0
-pin11
-Text GLabel 5150 7200 0    50   Input ~ 0
-pin14
-Text GLabel 2250 3300 2    50   Input ~ 0
-pin7
 Wire Wire Line
 	2150 3300 2200 3300
-Text GLabel 2750 3300 0    50   Input ~ 0
-pin6
 $Comp
 L Device:R R4
@@
 F 0 "C2" V 2698 2400 50  0000 C CNN
 F 1 "2.2nF" V 2789 2400 50  0000 C CNN
-F 2 "" H 2988 2250 50  0001 C CNN
+F 2 "libraries:C_Flat_L7.2_H6.5" H 2988 2250 50  0001 C CNN
 F 3 "~" H 2950 2400 50  0001 C CNN
 	1    2950 2400
@@
 	0    -1   -1   0
 $EndComp
-Text GLabel 3500 2400 2    50   Input ~ 0
-pin9
-Text GLabel 4050 2400 0    50   Input ~ 0
-pin10
 $Comp
 L Device:R_POT RV1
@@
 F 3 "~" H 4100 2200 50  0001 C CNN
 	1    4100 2200
-	0    -1   1    0
+	0    1    1    0
 $EndComp
 $Comp
@@
 F 0 "C4" V 4448 2400 50  0000 C CNN
 F 1 "470nF" V 4539 2400 50  0000 C CNN
-F 2 "" H 4738 2250 50  0001 C CNN
+F 2 "libraries:C_Flat_L7.2_H6.5" H 4738 2250 50  0001 C CNN
 F 3 "~" H 4700 2400 50  0001 C CNN
 	1    4700 2400
 	0    1    1    0
 $EndComp
-Text GLabel 4950 2400 2    50   Input ~ 0
-pin11
-Text GLabel 5550 2400 0    50   Input ~ 0
-pin12
 $Comp
 L Device:R R8
@@
 F 0 "C5" V 5548 2400 50  0000 C CNN
 F 1 "100nF" V 5639 2400 50  0000 C CNN
-F 2 "" H 5838 2250 50  0001 C CNN
+F 2 "libraries:C_Flat_L7.2_H6.5" H 5838 2250 50  0001 C CNN
 F 3 "~" H 5800 2400 50  0001 C CNN
 	1    5800 2400
@@
 F 0 "C6" H 6100 2600 50  0000 C CNN
 F 1 "1.5nF" H 6100 2700 50  0000 C CNN
-F 2 "" H 6338 2450 50  0001 C CNN
+F 2 "libraries:C_Flat_L7.2_H6.5" H 6338 2450 50  0001 C CNN
 F 3 "~" H 6300 2600 50  0001 C CNN
 	1    6300 2600
@@
 F 3 "~" H 6800 2400 50  0001 C CNN
 	1    6800 2400
-	0    1    1    0
-$EndComp
-Text GLabel 7050 2400 2    50   Input ~ 0
-pin14
+	0    -1   1    0
+$EndComp
 Wire Wire Line
 	6950 2400 7000 2400
@@
 Wire Wire Line
 	7000 2400 7050 2400
-Text GLabel 7650 2400 0    50   Input ~ 0
-pin15
 $Comp
 L Device:C C7
@@
 F 0 "C7" V 7098 2200 50  0000 C CNN
 F 1 "150pF" V 7189 2200 50  0000 C CNN
-F 2 "" H 7388 2050 50  0001 C CNN
+F 2 "Capacitor_THT:C_Axial_L5.1mm_D3.1mm_P10.00mm_Horizontal" H 7388 2050 50  0001 C CNN
 F 3 "~" H 7350 2200 50  0001 C CNN
 	1    7350 2200
@@
 F 0 "C9" V 7648 2400 50  0000 C CNN
 F 1 "100nF" V 7739 2400 50  0000 C CNN
-F 2 "" H 7938 2250 50  0001 C CNN
+F 2 "libraries:C_Flat_L7.2_H6.5" H 7938 2250 50  0001 C CNN
 F 3 "~" H 7900 2400 50  0001 C CNN
 	1    7900 2400
@@
 	0    -1   -1   0
 $EndComp
-Text GLabel 8450 2400 2    50   Input ~ 0
-pin3
-Text GLabel 8950 2400 0    50   Input ~ 0
-pin2
 $Comp
 L Device:C C10
@@
 F 0 "C10" H 8850 2650 50  0000 C CNN
 F 1 "100nF" H 8850 2750 50  0000 C CNN
-F 2 "" H 9088 2500 50  0001 C CNN
+F 2 "libraries:C_Flat_L7.2_H6.5" H 9088 2500 50  0001 C CNN
 F 3 "~" H 9050 2650 50  0001 C CNN
 	1    9050 2650
@@
 F 3 "~" H 9050 2950 50  0001 C CNN
 	1    9050 2950
-	1    0    0    1
+	1    0    0    -1
 $EndComp
 Text Label 9300 2950 0    50   ~ 0
@@
 F 0 "C8" V 7400 3300 50  0000 C CNN
 F 1 "100nF" V 7500 3300 50  0000 C CNN
-F 2 "" H 7688 3150 50  0001 C CNN
+F 2 "libraries:C_Flat_L7.2_H6.5" H 7688 3150 50  0001 C CNN
 F 3 "~" H 7650 3300 50  0001 C CNN
 	1    7650 3300
@@
 	8400 3300 8100 3300
 NoConn ~ 6550 6800
-Text GLabel 5950 5700 1    50   Input ~ 0
-pin8
-Text GLabel 5750 5700 1    50   Input ~ 0
-pin5
 $Comp
 L power:GND #PWR0106
@@
 F 0 "C3" H 3418 5996 50  0000 L CNN
 F 1 "100uF" H 3418 5905 50  0000 L CNN
-F 2 "" H 3338 5800 50  0001 C CNN
+F 2 "Capacitor_THT:CP_Axial_L10.0mm_D6.0mm_P15.00mm_Horizontal" H 3338 5800 50  0001 C CNN
 F 3 "~" H 3300 5950 50  0001 C CNN
 	1    3300 5950
 	1    0    0    -1
 $EndComp
-Text GLabel 3400 5700 2    50   Input ~ 0
-pin1
 Wire Wire Line
 	3200 5700 3300 5700
@@
 	1    0    0    -1
 $EndComp
+Text Label 5150 6800 2    50   ~ 0
+pin5
+Text Label 5750 5700 1    50   ~ 0
+pin5
+Text Label 6550 7400 0    50   ~ 0
+pin8
+Text Label 6550 7200 0    50   ~ 0
+pin15
+Text Label 6550 7100 0    50   ~ 0
+pin12
+Text Label 6550 7000 0    50   ~ 0
+pin10
+Text Label 6550 6900 0    50   ~ 0
+pin6
+Text Label 6550 6700 0    50   ~ 0
+pin2
+Text Label 6550 6500 0    50   ~ 0
+pin1
+Text Label 5150 6700 2    50   ~ 0
+pin3
+Text Label 5150 6900 2    50   ~ 0
+pin7
+Text Label 5150 7000 2    50   ~ 0
+pin9
+Text Label 5150 7100 2    50   ~ 0
+pin11
+Text Label 5150 7200 2    50   ~ 0
+pin14
+Text Label 3400 5700 0    50   ~ 0
+pin1
+Text Label 2250 3300 0    50   ~ 0
+pin7
+Text Label 2750 3300 2    50   ~ 0
+pin6
+Text Label 4050 2400 2    50   ~ 0
+pin10
+Text Label 3500 2400 0    50   ~ 0
+pin9
+Text Label 4950 2400 0    50   ~ 0
+pin11
+Text Label 5550 2400 2    50   ~ 0
+pin12
+Text Label 7050 2400 0    50   ~ 0
+pin14
+Text Label 7650 2400 2    50   ~ 0
+pin15
+Text Label 8450 2400 0    50   ~ 0
+pin3
+Text Label 8950 2400 2    50   ~ 0
+pin2
+Text Label 5950 5700 1    50   ~ 0
+pin8
 $EndSCHEMATC
