File: ConsolePedalDelay/ConsolePedalDelay.sch (KiCad schematic (older format))
At the start: 55 parts, among them J1 Conn_02x25_Counter_Clockwise, U1 TL072, U2 PT2399, U3 L78L05_TO92

Commit message: Finished assigning footprints
Parts:
- C1, C10, C11, C12, C15, C16, C18, C19, C6, C7, C8, C9: footprint (none) -> libraries:C_Flat_L7.2_H6.5
- C13, C14, C4, C5: footprint (none) -> libraries:CP_Radial_D5.0mm_P2.00mm
- C17, C21, C22: footprint (none) -> libraries:CP_Radial_D6.3mm_P2.50mm
- C2, C3: footprint (none) -> Capacitor_THT:C_Axial_L3.8mm_D2.6mm_P7.50mm_Horizontal
- C20: footprint (none) -> libraries:CP_Radial_D6.3mm_P2.00mm
Changed lines of the file:
@@
 F 0 "C1" V 1898 1200 50  0000 C CNN
 F 1 "22nF" V 1989 1200 50  0000 C CNN
-F 2 "" H 2188 1050 50  0001 C CNN
+F 2 "libraries:C_Flat_L7.2_H6.5" H 2188 1050 50  0001 C CNN
 F 3 "~" H 2150 1200 50  0001 C CNN
 	1    2150 1200
@@
 F 0 "C2" V 2850 1850 50  0000 C CNN
 F 1 "47pF" V 2750 1850 50  0000 C CNN
-F 2 "" H 3038 1700 50  0001 C CNN
+F 2 "Capacitor_THT:C_Axial_L3.8mm_D2.6mm_P7.50mm_Horizontal" H 3038 1700 50  0001 C CNN
 F 3 "~" H 3000 1850 50  0001 C CNN
 	1    3000 1850
@@
 F 0 "C5" H 3718 1546 50  0000 L CNN
 F 1 "1uF" H 3718 1455 50  0000 L CNN
-F 2 "" H 3638 1350 50  0001 C CNN
+F 2 "libraries:CP_Radial_D5.0mm_P2.00mm" H 3638 1350 50  0001 C CNN
 F 3 "~" H 3600 1500 50  0001 C CNN
 	1    3600 1500
@@
 F 0 "C4" V 5105 1000 50  0000 C CNN
 F 1 "1uF" V 5014 1000 50  0000 C CNN
-F 2 "" H 4888 850 50  0001 C CNN
+F 2 "libraries:CP_Radial_D5.0mm_P2.00mm" H 4888 850 50  0001 C CNN
 F 3 "~" H 4850 1000 50  0001 C CNN
 	1    4850 1000
@@
 F 0 "C6" H 2850 2450 50  0000 C CNN
 F 1 "4.7nF" H 2800 2350 50  0000 C CNN
-F 2 "" H 3038 2300 50  0001 C CNN
+F 2 "libraries:C_Flat_L7.2_H6.5" H 3038 2300 50  0001 C CNN
 F 3 "~" H 3000 2450 50  0001 C CNN
 	1    3000 2450
@@
 F 0 "C7" H 3150 3250 50  0000 C CNN
 F 1 "2.2nF" H 3100 3150 50  0000 C CNN
-F 2 "" H 3338 3050 50  0001 C CNN
+F 2 "libraries:C_Flat_L7.2_H6.5" H 3338 3050 50  0001 C CNN
 F 3 "~" H 3300 3200 50  0001 C CNN
 	1    3300 3200
@@
 F 0 "C11" V 3900 2700 50  0000 C CNN
 F 1 "22nF" V 4000 2750 50  0000 C CNN
-F 2 "" H 4188 2600 50  0001 C CNN
+F 2 "libraries:C_Flat_L7.2_H6.5" H 4188 2600 50  0001 C CNN
 F 3 "~" H 4150 2750 50  0001 C CNN
 	1    4150 2750
@@
 F 0 "C3" V 4200 1600 50  0000 C CNN
 F 1 "100pF" V 4300 1650 50  0000 C CNN
-F 2 "" H 4488 1500 50  0001 C CNN
+F 2 "Capacitor_THT:C_Axial_L3.8mm_D2.6mm_P7.50mm_Horizontal" H 4488 1500 50  0001 C CNN
 F 3 "~" H 4450 1650 50  0001 C CNN
 	1    4450 1650
@@
 F 0 "C14" V 4505 2200 50  0000 C CNN
 F 1 "1uF" V 4414 2200 50  0000 C CNN
-F 2 "" H 4288 2050 50  0001 C CNN
+F 2 "libraries:CP_Radial_D5.0mm_P2.00mm" H 4288 2050 50  0001 C CNN
 F 3 "~" H 4250 2200 50  0001 C CNN
 	1    4250 2200
@@
 F 0 "C8" H 3150 3850 50  0000 C CNN
 F 1 "2.2nF" H 3100 3750 50  0000 C CNN
-F 2 "" H 3338 3650 50  0001 C CNN
+F 2 "libraries:C_Flat_L7.2_H6.5" H 3338 3650 50  0001 C CNN
 F 3 "~" H 3300 3800 50  0001 C CNN
 	1    3300 3800
@@
 F 0 "C12" H 4350 3850 50  0000 C CNN
 F 1 "10nF" H 4350 3750 50  0000 C CNN
-F 2 "" H 4588 3650 50  0001 C CNN
+F 2 "libraries:C_Flat_L7.2_H6.5" H 4588 3650 50  0001 C CNN
 F 3 "~" H 4550 3800 50  0001 C CNN
 	1    4550 3800
@@
 F 0 "C13" V 5305 3650 50  0000 C CNN
 F 1 "1uF" V 5214 3650 50  0000 C CNN
-F 2 "" H 5088 3500 50  0001 C CNN
+F 2 "libraries:CP_Radial_D5.0mm_P2.00mm" H 5088 3500 50  0001 C CNN
 F 3 "~" H 5050 3650 50  0001 C CNN
 	1    5050 3650
@@
 F 0 "C15" H 5000 4350 50  0000 C CNN
 F 1 "47nF" H 5000 4250 50  0000 C CNN
-F 2 "" H 5238 4150 50  0001 C CNN
+F 2 "libraries:C_Flat_L7.2_H6.5" H 5238 4150 50  0001 C CNN
 F 3 "~" H 5200 4300 50  0001 C CNN
 	1    5200 4300
@@
 F 0 "C9" H 3050 4450 50  0000 C CNN
 F 1 "100nF" H 3050 4350 50  0000 C CNN
-F 2 "" H 3338 4250 50  0001 C CNN
+F 2 "libraries:C_Flat_L7.2_H6.5" H 3338 4250 50  0001 C CNN
 F 3 "~" H 3300 4400 50  0001 C CNN
 	1    3300 4400
@@
 F 0 "C16" H 3750 4750 50  0000 C CNN
 F 1 "15nF" H 3750 4650 50  0000 C CNN
-F 2 "" H 3988 4550 50  0001 C CNN
+F 2 "libraries:C_Flat_L7.2_H6.5" H 3988 4550 50  0001 C CNN
 F 3 "~" H 3950 4700 50  0001 C CNN
 	1    3950 4700
@@
 F 0 "C10" H 3100 5050 50  0000 C CNN
 F 1 "100nF" H 3100 4950 50  0000 C CNN
-F 2 "" H 3338 4850 50  0001 C CNN
+F 2 "libraries:C_Flat_L7.2_H6.5" H 3338 4850 50  0001 C CNN
 F 3 "~" H 3300 5000 50  0001 C CNN
 	1    3300 5000
@@
 F 0 "C19" V 1750 4750 50  0000 C CNN
 F 1 "100nF" V 1850 4750 50  0000 C CNN
-F 2 "" H 1988 4400 50  0001 C CNN
+F 2 "libraries:C_Flat_L7.2_H6.5" H 1988 4400 50  0001 C CNN
 F 3 "~" H 1950 4550 50  0001 C CNN
 	1    1950 4550
@@
 F 0 "C18" V 1750 4450 50  0000 C CNN
 F 1 "100nF" V 1850 4450 50  0000 C CNN
-F 2 "" H 1988 4100 50  0001 C CNN
+F 2 "libraries:C_Flat_L7.2_H6.5" H 1988 4100 50  0001 C CNN
 F 3 "~" H 1950 4250 50  0001 C CNN
 	1    1950 4250
@@
 F 0 "C17" V 1695 3950 50  0000 C CNN
 F 1 "47uF" V 1786 3950 50  0000 C CNN
-F 2 "" H 1988 3800 50  0001 C CNN
+F 2 "libraries:CP_Radial_D6.3mm_P2.50mm" H 1988 3800 50  0001 C CNN
 F 3 "~" H 1950 3950 50  0001 C CNN
 	1    1950 3950
@@
 F 0 "C20" H 2268 6096 50  0000 L CNN
 F 1 "100uF" H 2268 6005 50  0000 L CNN
-F 2 "" H 2188 5900 50  0001 C CNN
+F 2 "libraries:CP_Radial_D6.3mm_P2.00mm" H 2188 5900 50  0001 C CNN
 F 3 "~" H 2150 6050 50  0001 C CNN
 	1    2150 6050
@@
 F 0 "C21" H 3718 6246 50  0000 L CNN
 F 1 "47uF" H 3718 6155 50  0000 L CNN
-F 2 "" H 3638 6050 50  0001 C CNN
+F 2 "libraries:CP_Radial_D6.3mm_P2.50mm" H 3638 6050 50  0001 C CNN
 F 3 "~" H 3600 6200 50  0001 C CNN
 	1    3600 6200
@@
 F 0 "C22" H 4768 6146 50  0000 L CNN
 F 1 "47uF" H 4768 6055 50  0000 L CNN
-F 2 "" H 4688 5950 50  0001 C CNN
+F 2 "libraries:CP_Radial_D6.3mm_P2.50mm" H 4688 5950 50  0001 C CNN
 F 3 "~" H 4650 6100 50  0001 C CNN
 	1    4650 6100

Commit message: Still working on routing traces
Parts:
- C13, C14, C4, C5: footprint libraries:CP_Radial_D5.0mm_P2.00mm -> libraries:CP_Radial_D5.0mm_P2.00mm_L11.0mm
- C17, C21, C22: footprint libraries:CP_Radial_D6.3mm_P2.50mm -> libraries:CP_Radial_D6.3mm_P2.50mm_L7.0mm
- C20: footprint libraries:CP_Radial_D6.3mm_P2.00mm -> libraries:CP_Radial_D6.3mm_P2.00mm_L11.0mm
- U1: footprint Package_DIP:DIP-8_W7.62mm_Socket_LongPads -> Package_DIP:DIP-8_W7.62mm_Socket
- U2: footprint Package_DIP:DIP-16_W7.62mm_Socket_LongPads -> Package_DIP:DIP-16_W7.62mm_Socket
Changed lines of the file:
@@
 F 0 "U1" H 3000 1467 50  0000 C CNN
 F 1 "TL072" H 3000 1376 50  0000 C CNN
-F 2 "Package_DIP:DIP-8_W7.62mm_Socket_LongPads" H 3000 1100 50  0001 C CNN
+F 2 "Package_DIP:DIP-8_W7.62mm_Socket" H 3000 1100 50  0001 C CNN
 F 3 "http://www.ti.com/lit/ds/symlink/tl071.pdf" H 3000 1100 50  0001 C CNN
 	1    3000 1100
@@
 F 0 "U1" H 4350 1367 50  0000 C CNN
 F 1 "TL072" H 4350 1276 50  0000 C CNN
-F 2 "Package_DIP:DIP-8_W7.62mm_Socket_LongPads" H 4350 1000 50  0001 C CNN
+F 2 "Package_DIP:DIP-8_W7.62mm_Socket" H 4350 1000 50  0001 C CNN
 F 3 "http://www.ti.com/lit/ds/symlink/tl071.pdf" H 4350 1000 50  0001 C CNN
 	2    4350 1000
@@
 F 0 "U1" H 2708 6096 50  0000 L CNN
 F 1 "TL072" H 2708 6005 50  0000 L CNN
-F 2 "Package_DIP:DIP-8_W7.62mm_Socket_LongPads" H 2750 6050 50  0001 C CNN
+F 2 "Package_DIP:DIP-8_W7.62mm_Socket" H 2750 6050 50  0001 C CNN
 F 3 "http://www.ti.com/lit/ds/symlink/tl071.pdf" H 2750 6050 50  0001 C CNN
 	3    2750 6050
@@
 F 0 "C5" H 3718 1546 50  0000 L CNN
 F 1 "1uF" H 3718 1455 50  0000 L CNN
-F 2 "libraries:CP_Radial_D5.0mm_P2.00mm" H 3638 1350 50  0001 C CNN
+F 2 "libraries:CP_Radial_D5.0mm_P2.00mm_L11.0mm" H 3638 1350 50  0001 C CNN
 F 3 "~" H 3600 1500 50  0001 C CNN
 	1    3600 1500
@@
 F 0 "C4" V 5105 1000 50  0000 C CNN
 F 1 "1uF" V 5014 1000 50  0000 C CNN
-F 2 "libraries:CP_Radial_D5.0mm_P2.00mm" H 4888 850 50  0001 C CNN
+F 2 "libraries:CP_Radial_D5.0mm_P2.00mm_L11.0mm" H 4888 850 50  0001 C CNN
 F 3 "~" H 4850 1000 50  0001 C CNN
 	1    4850 1000
@@
 F 0 "U2" H 9300 2117 50  0000 C CNN
 F 1 "PT2399" H 9300 2026 50  0000 C CNN
-F 2 "Package_DIP:DIP-16_W7.62mm_Socket_LongPads" H 9300 950 50  0001 C CNN
+F 2 "Package_DIP:DIP-16_W7.62mm_Socket" H 9300 950 50  0001 C CNN
 F 3 "http://sound.westhost.com/pt2399.pdf" H 9300 950 50  0001 C CNN
 	1    9300 1350
@@
 F 0 "C14" V 4505 2200 50  0000 C CNN
 F 1 "1uF" V 4414 2200 50  0000 C CNN
-F 2 "libraries:CP_Radial_D5.0mm_P2.00mm" H 4288 2050 50  0001 C CNN
+F 2 "libraries:CP_Radial_D5.0mm_P2.00mm_L11.0mm" H 4288 2050 50  0001 C CNN
 F 3 "~" H 4250 2200 50  0001 C CNN
 	1    4250 2200
@@
 F 0 "C13" V 5305 3650 50  0000 C CNN
 F 1 "1uF" V 5214 3650 50  0000 C CNN
-F 2 "libraries:CP_Radial_D5.0mm_P2.00mm" H 5088 3500 50  0001 C CNN
+F 2 "libraries:CP_Radial_D5.0mm_P2.00mm_L11.0mm" H 5088 3500 50  0001 C CNN
 F 3 "~" H 5050 3650 50  0001 C CNN
 	1    5050 3650
@@
 F 0 "C17" V 1695 3950 50  0000 C CNN
 F 1 "47uF" V 1786 3950 50  0000 C CNN
-F 2 "libraries:CP_Radial_D6.3mm_P2.50mm" H 1988 3800 50  0001 C CNN
+F 2 "libraries:CP_Radial_D6.3mm_P2.50mm_L7.0mm" H 1988 3800 50  0001 C CNN
 F 3 "~" H 1950 3950 50  0001 C CNN
 	1    1950 3950
@@
 F 0 "C20" H 2268 6096 50  0000 L CNN
 F 1 "100uF" H 2268 6005 50  0000 L CNN
-F 2 "libraries:CP_Radial_D6.3mm_P2.00mm" H 2188 5900 50  0001 C CNN
+F 2 "libraries:CP_Radial_D6.3mm_P2.00mm_L11.0mm" H 2188 5900 50  0001 C CNN
 F 3 "~" H 2150 6050 50  0001 C CNN
 	1    2150 6050
@@
 F 0 "C21" H 3718 6246 50  0000 L CNN
 F 1 "47uF" H 3718 6155 50  0000 L CNN
-F 2 "libraries:CP_Radial_D6.3mm_P2.50mm" H 3638 6050 50  0001 C CNN
+F 2 "libraries:CP_Radial_D6.3mm_P2.50mm_L7.0mm" H 3638 6050 50  0001 C CNN
 F 3 "~" H 3600 6200 50  0001 C CNN
 	1    3600 6200
@@
 F 0 "C22" H 4768 6146 50  0000 L CNN
 F 1 "47uF" H 4768 6055 50  0000 L CNN
-F 2 "libraries:CP_Radial_D6.3mm_P2.50mm" H 4688 5950 50  0001 C CNN
+F 2 "libraries:CP_Radial_D6.3mm_P2.50mm_L7.0mm" H 4688 5950 50  0001 C CNN
 F 3 "~" H 4650 6100 50  0001 C CNN
 	1    4650 6100
