File: ConsolePedalDelay/ConsolePedalDelay.kicad_pcb (KiCad board)
At the start: 2 copper layers, 100 x 60 mm, 55 parts, among them J1 Conn_02x25_Counter_Clockwise, U1 TL072, U2 PT2399, U3 L78L05_TO92

Commit message: Still working on routing traces
Parts:
- C1, C10, C11, C12, C19, C6, C7, C9: moved to B.Cu
- C13, C14, C4, C5: footprint libraries:CP_Radial_D5.0mm_P2.00mm -> libraries:CP_Radial_D5.0mm_P2.00mm_L11.0mm
- C17, C21, C22: footprint libraries:CP_Radial_D6.3mm_P2.50mm -> libraries:CP_Radial_D6.3mm_P2.50mm_L7.0mm
- C20: footprint libraries:CP_Radial_D6.3mm_P2.00mm -> libraries:CP_Radial_D6.3mm_P2.00mm_L11.0mm
- U1: footprint Package_DIP:DIP-8_W7.62mm_Socket_LongPads -> Package_DIP:DIP-8_W7.62mm_Socket
- U2: footprint Package_DIP:DIP-16_W7.62mm_Socket_LongPads -> Package_DIP:DIP-16_W7.62mm_Socket
- moved C7 109.2 mm to (102.4, 102.6), turned to 180 degrees
- moved C8 107.7 mm to (94.2, 110.7), turned to 180 degrees
- moved C21 106.1 mm to (167.9, 109.0), turned to 180 degrees
- moved C19 96.5 mm to (110.5, 102.6), turned to 180 degrees
- moved R15 96.2 mm to (86.6, 81.8)
- moved C17 94.8 mm to (109.2, 111.3), turned to 180 degrees
- moved C9 92.0 mm to (94.2, 102.6), turned to 180 degrees
- moved C3 85.8 mm to (111.3, 91.2)
- moved C16 83.2 mm to (177.3, 108.5), turned to 180 degrees
- moved U2 81.7 mm to (128.9, 92.7)
- moved C13 78.2 mm to (159.3, 112.3), turned to 180 degrees
- moved R18 77.2 mm to (113.3, 85.1)
- moved C18 76.2 mm to (94.2, 98.8), turned to 180 degrees
- moved R17 75.8 mm to (113.3, 75.2)
- moved R9 74.3 mm to (96.8, 75.2), turned to 180 degrees
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Routing:
- net Net-(C3-Pad1): track 0.00 -> 116.8 mm, vias 0 -> 1
- net Net-(C6-Pad1): track 0.00 -> 112.6 mm, vias 0 -> 2
- net /LEDPower: track 54.1 -> 126.8 mm
- net /VREF: track 0.00 -> 65.5 mm
- net /Input: track 71.6 -> 131.4 mm
- net /Output: track 66.0 -> 121.6 mm, vias 2 -> 3
- net Net-(C1-Pad1): track 0.00 -> 54.7 mm
- net /pin11: track 0.00 -> 54.3 mm, vias 0 -> 1
- net Net-(C2-Pad2): track 0.00 -> 47.5 mm
- net Net-(C16-Pad2): track 0.00 -> 47.2 mm
- net /pin6: track 0.00 -> 41.1 mm
- net Net-(C3-Pad2): track 0.00 -> 40.9 mm
- net +9V: track 60.1 -> 99.2 mm, vias 2 -> 3
- net /pin7: track 0.00 -> 38.3 mm
- net Net-(C15-Pad2): track 0.00 -> 37.7 mm
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Other:
- board text added: "Console Pedal Delay V1.0"
- board text removed: "Console Pedal Shake V1.0"

Commit message: Minor changes. Still not done with traces
Parts:
- moved R2 0.17 mm to (141.0, 71.8)
Routing:
- net Net-(C14-Pad1): track 0.00 -> 103.5 mm, vias 0 -> 1
- net /VREF: track 65.5 -> 161.6 mm
- net Net-(C13-Pad2): track 0.00 -> 81.5 mm, vias 0 -> 1
- net Net-(C2-Pad1): track 22.4 -> 102.1 mm
- net Net-(C5-Pad2): track 0.00 -> 74.3 mm, vias 0 -> 1
- net Net-(C20-Pad1): track 23.4 -> 95.1 mm, vias 0 -> 1
- net /pin13: track 0.00 -> 62.0 mm, vias 0 -> 1
- net Net-(C4-Pad2): track 0.00 -> 56.8 mm, vias 0 -> 1
- net /pin14: track 3.30 -> 50.9 mm, vias 0 -> 1
- net Net-(C16-Pad2): track 47.2 -> 88.5 mm
- net /pin10: track 0.00 -> 37.7 mm, vias 0 -> 2
- net /5V: track 0.00 -> 37.3 mm, vias 0 -> 1
- net /pin9: track 0.00 -> 34.1 mm
- net Net-(C2-Pad2): track 47.5 -> 80.2 mm, vias 0 -> 1
- net /pin2: track 0.00 -> 29.3 mm
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
Commit message: Finalized board and plotted gerbers. Had to use a 4 layer board for the first time
Routing:
- net Net-(C2-Pad2): track 80.2 -> 160.2 mm
- net Net-(C12-Pad2): track 13.8 -> 87.5 mm
- net /pin12: track 36.6 -> 82.3 mm
- net /pin16: track 25.1 -> 70.5 mm
- net /pin15: track 33.7 -> 78.0 mm
- net /pin13: track 62.0 -> 102.0 mm
- net /5V: track 37.3 -> 73.8 mm
- net /pin14: track 50.9 -> 87.1 mm
- net Net-(C3-Pad2): track 40.9 -> 75.1 mm
- net /pin4: track 0.00 -> 34.0 mm
- net Net-(D1-Pad1): track 0.00 -> 32.4 mm
- net Net-(D2-Pad1): track 15.0 -> 40.5 mm
- net GND: vias 4 -> 8
- added copper zone on In1.Cu, net GND
- added copper zone on In2.Cu, net GND
Other:
- copper layers 2 -> 4
