File: ConsolePedalDS1/ConsolePedalDS1.sch (KiCad schematic (older format))
At the start: 62 parts, among them J1 Conn_02x25_Counter_Clockwise, Q1 2N5088, Q2 2N5088, U1 TL072

Commit message: Minor changes
Parts:
- Q1, Q2: footprint (none) -> Package_TO_SOT_THT:TO-92_Inline
- Q3: renamed from Q?; footprint (none) -> Package_TO_SOT_THT:TO-92_Inline
- U1: footprint (none) -> Package_DIP:DIP-8_W7.62mm_Socket
- gave numbers to parts that had none: 2
- renumbered D1 to D5, D2 to D8
Changed lines of the file:
@@
 LEDPower
 $Comp
-L Device:LED D?
+L Device:LED D7
 U 1 1 5FA93C7E
 P 10150 5850
-F 0 "D?" H 10143 5595 50  0000 C CNN
+F 0 "D7" H 10143 5595 50  0000 C CNN
 F 1 "LED" H 10143 5686 50  0000 C CNN
 F 2 "LED_THT:LED_D5.0mm" H 10150 5850 50  0001 C CNN
@@
 LEDPower
 $Comp
-L Device:LED D2
+L Device:LED D8
 U 1 1 5FA94A27
 P 10150 6050
-F 0 "D2" H 10150 6150 50  0000 C CNN
+F 0 "D8" H 10150 6150 50  0000 C CNN
 F 1 "LED" H 10150 6250 50  0000 C CNN
 F 2 "LED_THT:LED_D5.0mm" H 10150 6050 50  0001 C CNN
@@
 	10000 5850 10000 5950
 $Comp
-L Device:R R?
+L Device:R R28
 U 1 1 5FA964BB
 P 10600 5950
-F 0 "R?" H 10670 5996 50  0000 L CNN
+F 0 "R28" H 10670 5996 50  0000 L CNN
 F 1 "100K" H 10670 5905 50  0000 L CNN
 F 2 "Resistor_THT:R_Axial_DIN0207_L6.3mm_D2.5mm_P10.16mm_Horizontal" V 10530 5950 50  0001 C CNN
@@
 F 0 "Q1" H 1940 1946 50  0000 L CNN
 F 1 "2N5088" H 1940 1855 50  0000 L CNN
-F 2 "" H 1950 2000 50  0001 C CNN
+F 2 "Package_TO_SOT_THT:TO-92_Inline" H 1950 2000 50  0001 C CNN
 F 3 "~" H 1750 1900 50  0001 C CNN
 	1    1750 1900
@@
 	1500 1900 1550 1900
 $Comp
-L power:+9V #PWR?
+L power:+9V #PWR0103
 U 1 1 60B4020B
 P 1850 1000
-F 0 "#PWR?" H 1850 850 50  0001 C CNN
+F 0 "#PWR0103" H 1850 850 50  0001 C CNN
 F 1 "+9V" H 1750 1150 50  0000 L CNN
 F 2 "" H 1850 1000 50  0001 C CNN
@@
 Connection ~ 1850 2200
 $Comp
-L power:GND #PWR?
+L power:GND #PWR0104
 U 1 1 60B47089
 P 1850 2600
-F 0 "#PWR?" H 1850 2350 50  0001 C CNN
+F 0 "#PWR0104" H 1850 2350 50  0001 C CNN
 F 1 "GND" H 1855 2427 50  0000 C CNN
 F 2 "" H 1850 2600 50  0001 C CNN
@@
 $EndComp
 $Comp
-L power:GND #PWR?
+L power:GND #PWR0105
 U 1 1 60B47A26
 P 800 2250
-F 0 "#PWR?" H 800 2000 50  0001 C CNN
+F 0 "#PWR0105" H 800 2000 50  0001 C CNN
 F 1 "GND" H 805 2077 50  0000 C CNN
 F 2 "" H 800 2250 50  0001 C CNN
@@
 F 0 "Q2" H 3490 2246 50  0000 L CNN
 F 1 "2N5088" H 3490 2155 50  0000 L CNN
-F 2 "" H 3500 2300 50  0001 C CNN
+F 2 "Package_TO_SOT_THT:TO-92_Inline" H 3500 2300 50  0001 C CNN
 F 3 "~" H 3300 2200 50  0001 C CNN
 	1    3300 2200
@@
 $EndComp
 $Comp
-L power:GND #PWR?
+L power:GND #PWR0106
 U 1 1 60B51751
 P 3400 2700
-F 0 "#PWR?" H 3400 2450 50  0001 C CNN
+F 0 "#PWR0106" H 3400 2450 50  0001 C CNN
 F 1 "GND" H 3405 2527 50  0000 C CNN
 F 2 "" H 3400 2700 50  0001 C CNN
@@
 	3400 1850 3400 2000
 $Comp
-L power:GND #PWR?
+L power:GND #PWR0107
 U 1 1 60B594E9
 P 3100 2700
-F 0 "#PWR?" H 3100 2450 50  0001 C CNN
+F 0 "#PWR0107" H 3100 2450 50  0001 C CNN
 F 1 "GND" H 3105 2527 50  0000 C CNN
 F 2 "" H 3100 2700 50  0001 C CNN
@@
 Connection ~ 3400 1850
 $Comp
-L power:+9V #PWR?
+L power:+9V #PWR0108
 U 1 1 60B6F7CA
 P 3400 1000
-F 0 "#PWR?" H 3400 850 50  0001 C CNN
+F 0 "#PWR0108" H 3400 850 50  0001 C CNN
 F 1 "+9V" H 3300 1150 50  0000 L CNN
 F 2 "" H 3400 1000 50  0001 C CNN
@@
 F 0 "U1" H 4600 2317 50  0000 C CNN
 F 1 "TL072" H 4600 2226 50  0000 C CNN
-F 2 "" H 4600 1950 50  0001 C CNN
+F 2 "Package_DIP:DIP-8_W7.62mm_Socket" H 4600 1950 50  0001 C CNN
 F 3 "http://www.ti.com/lit/ds/symlink/tl071.pdf" H 4600 1950 50  0001 C CNN
 	1    4600 1950
@@
 F 0 "U1" H 5800 1717 50  0000 C CNN
 F 1 "TL072" H 5800 1626 50  0000 C CNN
-F 2 "" H 5800 1350 50  0001 C CNN
+F 2 "Package_DIP:DIP-8_W7.62mm_Socket" H 5800 1350 50  0001 C CNN
 F 3 "http://www.ti.com/lit/ds/symlink/tl071.pdf" H 5800 1350 50  0001 C CNN
 	2    5800 1350
@@
 F 0 "U1" H 9108 5996 50  0000 L CNN
 F 1 "TL072" H 9108 5905 50  0000 L CNN
-F 2 "" H 9150 5950 50  0001 C CNN
+F 2 "Package_DIP:DIP-8_W7.62mm_Socket" H 9150 5950 50  0001 C CNN
 F 3 "http://www.ti.com/lit/ds/symlink/tl071.pdf" H 9150 5950 50  0001 C CNN
 	3    9150 5950
@@
 $EndComp
 $Comp
-L power:+9V #PWR?
+L power:+9V #PWR0109
 U 1 1 60B858D6
 P 9050 5650
-F 0 "#PWR?" H 9050 5500 50  0001 C CNN
+F 0 "#PWR0109" H 9050 5500 50  0001 C CNN
 F 1 "+9V" H 9000 5800 50  0000 L CNN
 F 2 "" H 9050 5650 50  0001 C CNN
@@
 $EndComp
 $Comp
-L power:GND #PWR?
+L power:GND #PWR0110
 U 1 1 60B87247
 P 9050 6250
-F 0 "#PWR?" H 9050 6000 50  0001 C CNN
+F 0 "#PWR0110" H 9050 6000 50  0001 C CNN
 F 1 "GND" H 9055 6077 50  0000 C CNN
 F 2 "" H 9050 6250 50  0001 C CNN
@@
 Connection ~ 4150 1850
 $Comp
-L power:GND #PWR?
+L power:GND #PWR0111
 U 1 1 60B98F6A
 P 4150 2700
-F 0 "#PWR?" H 4150 2450 50  0001 C CNN
+F 0 "#PWR0111" H 4150 2450 50  0001 C CNN
 F 1 "GND" H 4155 2527 50  0000 C CNN
 F 2 "" H 4150 2700 50  0001 C CNN
@@
 $EndComp
 $Comp
-L power:GND #PWR?
+L power:GND #PWR0112
 U 1 1 60BAD820
 P 6100 2950
-F 0 "#PWR?" H 6100 2700 50  0001 C CNN
+F 0 "#PWR0112" H 6100 2700 50  0001 C CNN
 F 1 "GND" H 6105 2777 50  0000 C CNN
 F 2 "" H 6100 2950 50  0001 C CNN
@@
 	6100 1050 6100 1350
 $Comp
-L power:+9V #PWR?
+L power:+9V #PWR0113
 U 1 1 60BC1BD7
 P 6100 750
-F 0 "#PWR?" H 6100 600 50  0001 C CNN
+F 0 "#PWR0113" H 6100 600 50  0001 C CNN
 F 1 "+9V" H 6000 900 50  0000 L CNN
 F 2 "" H 6100 750 50  0001 C CNN
@@
 $EndComp
 $Comp
-L Diode:1N4148 D1
+L Diode:1N4148 D5
 U 1 1 60BE6E66
 P 7500 1450
-F 0 "D1" H 7550 1550 50  0000 R CNN
+F 0 "D5" H 7550 1550 50  0000 R CNN
 F 1 "1N4148" H 7600 1350 50  0000 R CNN
 F 2 "Diode_THT:D_DO-35_SOD27_P7.62mm_Horizontal" H 7500 1275 50  0001 C CNN
@@
 Connection ~ 8250 1800
 $Comp
-L Device:Q_NPN_EBC Q?
+L Device:Q_NPN_EBC Q3
 U 1 1 60C82E8C
 P 3800 4050
-F 0 "Q?" H 3990 4096 50  0000 L CNN
+F 0 "Q3" H 3990 4096 50  0000 L CNN
 F 1 "2N5088" H 3990 4005 50  0000 L CNN
-F 2 "" H 4000 4150 50  0001 C CNN
+F 2 "Package_TO_SOT_THT:TO-92_Inline" H 4000 4150 50  0001 C CNN
 F 3 "~" H 3800 4050 50  0001 C CNN
 	1    3800 4050
@@
 Connection ~ 3500 4050
 $Comp
-L power:+9V #PWR?
+L power:+9V #PWR0114
 U 1 1 60C88D36
 P 3900 3650
-F 0 "#PWR?" H 3900 3500 50  0001 C CNN
+F 0 "#PWR0114" H 3900 3500 50  0001 C CNN
 F 1 "+9V" H 3800 3800 50  0000 L CNN
 F 2 "" H 3900 3650 50  0001 C CNN
@@
 $EndComp
 $Comp
-L power:GND #PWR?
+L power:GND #PWR0115
 U 1 1 60C8F58C
 P 3900 4650
-F 0 "#PWR?" H 3900 4400 50  0001 C CNN
+F 0 "#PWR0115" H 3900 4400 50  0001 C CNN
 F 1 "GND" H 3905 4477 50  0000 C CNN
 F 2 "" H 3900 4650 50  0001 C CNN
@@
 	5000 4300 4900 4300
 $Comp
-L power:GND #PWR?
+L power:GND #PWR0116
 U 1 1 60CA3648
 P 5000 4650
-F 0 "#PWR?" H 5000 4400 50  0001 C CNN
+F 0 "#PWR0116" H 5000 4400 50  0001 C CNN
 F 1 "GND" H 5005 4477 50  0000 C CNN
 F 2 "" H 5000 4650 50  0001 C CNN
@@
 Connection ~ 5000 4300
 $Comp
-L power:+9V #PWR?
+L power:+9V #PWR0117
 U 1 1 60CABCC6
 P 6550 4350
-F 0 "#PWR?" H 6550 4200 50  0001 C CNN
+F 0 "#PWR0117" H 6550 4200 50  0001 C CNN
 F 1 "+9V" H 6450 4500 50  0000 L CNN
 F 2 "" H 6550 4350 50  0001 C CNN
@@
 $EndComp
 $Comp
-L power:GND #PWR?
+L power:GND #PWR0118
 U 1 1 60CC51DC
 P 6550 4750
-F 0 "#PWR?" H 6550 4500 50  0001 C CNN
+F 0 "#PWR0118" H 6550 4500 50  0001 C CNN
 F 1 "GND" H 6555 4577 50  0000 C CNN
 F 2 "" H 6550 4750 50  0001 C CNN
@@
 $EndComp
 $Comp
-L power:GND #PWR?
+L power:GND #PWR0119
 U 1 1 60CC5A40
 P 7050 4750
-F 0 "#PWR?" H 7050 4500 50  0001 C CNN
+F 0 "#PWR0119" H 7050 4500 50  0001 C CNN
 F 1 "GND" H 7055 4577 50  0000 C CNN
 F 2 "" H 7050 4750 50  0001 C CNN
@@
 	7500 4800 7500 4750
 $Comp
-L power:GND #PWR?
+L power:GND #PWR0120
 U 1 1 60CD1437
 P 7500 5100
-F 0 "#PWR?" H 7500 4850 50  0001 C CNN
+F 0 "#PWR0120" H 7500 4850 50  0001 C CNN
 F 1 "GND" H 7505 4927 50  0000 C CNN
 F 2 "" H 7500 5100 50  0001 C CNN
@@
 	7500 4750 7500 4700
 $Comp
-L power:GND #PWR?
+L power:GND #PWR0121
 U 1 1 60CDAE0F
 P 7850 5100
-F 0 "#PWR?" H 7850 4850 50  0001 C CNN
+F 0 "#PWR0121" H 7850 4850 50  0001 C CNN
 F 1 "GND" H 7855 4927 50  0000 C CNN
 F 2 "" H 7850 5100 50  0001 C CNN

Commit message: Still working on routing traces
Parts:
- C1, C10, C11, C12, C2, C3, C5, C8, C9: footprint (none) -> libraries:C_Flat_L7.2_H6.5
- C13, C7: footprint (none) -> libraries:C_Flat_L7.2_H10
- C14: footprint (none) -> libraries:CP_Radial_D6.3mm_P2.50mm_L7.0mm
- C15: footprint (none) -> libraries:CP_Radial_D6.3mm_P2.00mm_L11.0mm
- C16, C6: footprint (none) -> Capacitor_THT:C_Axial_L3.8mm_D2.6mm_P7.50mm_Horizontal
- C4: footprint (none) -> Capacitor_THT:C_Axial_L5.1mm_D3.1mm_P7.50mm_Horizontal
- RV1, RV2, RV3: footprint (none) -> Potentiometer_THT:Potentiometer_Bourns_PTV09A-1_Single_Vertical
Changed lines of the file:
@@
 F 0 "C1" V 1048 1900 50  0000 C CNN
 F 1 "0.047uF" V 1139 1900 50  0000 C CNN
-F 2 "" H 1338 1750 50  0001 C CNN
+F 2 "libraries:C_Flat_L7.2_H6.5" H 1338 1750 50  0001 C CNN
 F 3 "~" H 1300 1900 50  0001 C CNN
 	1    1300 1900
@@
 F 0 "C2" V 1950 2200 50  0000 C CNN
 F 1 "0.47uF" V 1850 2200 50  0000 C CNN
-F 2 "" H 2138 2050 50  0001 C CNN
+F 2 "libraries:C_Flat_L7.2_H6.5" H 2138 2050 50  0001 C CNN
 F 3 "~" H 2100 2200 50  0001 C CNN
 	1    2100 2200
@@
 F 0 "C3" V 2550 2200 50  0000 C CNN
 F 1 "0.047uF" V 2450 2200 50  0000 C CNN
-F 2 "" H 2738 2050 50  0001 C CNN
+F 2 "libraries:C_Flat_L7.2_H6.5" H 2738 2050 50  0001 C CNN
 F 3 "~" H 2700 2200 50  0001 C CNN
 	1    2700 2200
@@
 F 0 "C4" V 3000 1500 50  0000 C CNN
 F 1 "220pF" V 3100 1500 50  0000 C CNN
-F 2 "" H 3288 1350 50  0001 C CNN
+F 2 "Capacitor_THT:C_Axial_L5.1mm_D3.1mm_P7.50mm_Horizontal" H 3288 1350 50  0001 C CNN
 F 3 "~" H 3250 1500 50  0001 C CNN
 	1    3250 1500
@@
 F 0 "C5" V 3300 1850 50  0000 C CNN
 F 1 "0.47uF" V 3400 1850 50  0000 C CNN
-F 2 "" H 3588 1700 50  0001 C CNN
+F 2 "libraries:C_Flat_L7.2_H6.5" H 3588 1700 50  0001 C CNN
 F 3 "~" H 3550 1850 50  0001 C CNN
 	1    3550 1850
@@
 F 0 "C6" V 5600 1950 50  0000 C CNN
 F 1 "100pF" V 5700 1950 50  0000 C CNN
-F 2 "" H 5888 1800 50  0001 C CNN
+F 2 "Capacitor_THT:C_Axial_L3.8mm_D2.6mm_P7.50mm_Horizontal" H 5888 1800 50  0001 C CNN
 F 3 "~" H 5850 1950 50  0001 C CNN
 	1    5850 1950
@@
 F 0 "RV1" H 6030 2154 50  0000 R CNN
 F 1 "Dist" H 6030 2245 50  0000 R CNN
-F 2 "" H 6100 2200 50  0001 C CNN
+F 2 "Potentiometer_THT:Potentiometer_Bourns_PTV09A-1_Single_Vertical" H 6100 2200 50  0001 C CNN
 F 3 "~" H 6100 2200 50  0001 C CNN
 	1    6100 2200
@@
 F 0 "C7" H 5900 2800 50  0000 C CNN
 F 1 "1uF" H 5900 2900 50  0000 C CNN
-F 2 "" H 6138 2650 50  0001 C CNN
+F 2 "libraries:C_Flat_L7.2_H10" H 6138 2650 50  0001 C CNN
 F 3 "~" H 6100 2800 50  0001 C CNN
 	1    6100 2800
@@
 F 0 "C8" V 6400 1350 50  0000 C CNN
 F 1 "0.47uF" V 6500 1350 50  0000 C CNN
-F 2 "" H 6688 1200 50  0001 C CNN
+F 2 "libraries:C_Flat_L7.2_H6.5" H 6688 1200 50  0001 C CNN
 F 3 "~" H 6650 1350 50  0001 C CNN
 	1    6650 1350
@@
 F 0 "C16" H 7050 1300 50  0000 C CNN
 F 1 "47pF" H 7100 1200 50  0000 C CNN
-F 2 "" H 7288 1150 50  0001 C CNN
+F 2 "Capacitor_THT:C_Axial_L3.8mm_D2.6mm_P7.50mm_Horizontal" H 7288 1150 50  0001 C CNN
 F 3 "~" H 7250 1300 50  0001 C CNN
 	1    7250 1300
@@
 F 0 "C9" H 8100 1500 50  0000 C CNN
 F 1 "0.01uF" H 8100 1400 50  0000 C CNN
-F 2 "" H 8288 1350 50  0001 C CNN
+F 2 "libraries:C_Flat_L7.2_H6.5" H 8288 1350 50  0001 C CNN
 F 3 "~" H 8250 1500 50  0001 C CNN
 	1    8250 1500
@@
 F 0 "C10" H 900 4250 50  0000 C CNN
 F 1 "0.022uF" H 900 4350 50  0000 C CNN
-F 2 "" H 1138 4100 50  0001 C CNN
+F 2 "libraries:C_Flat_L7.2_H6.5" H 1138 4100 50  0001 C CNN
 F 3 "~" H 1100 4250 50  0001 C CNN
 	1    1100 4250
@@
 F 0 "RV3" H 1781 4296 50  0000 R CNN
 F 1 "Tone" H 1781 4205 50  0000 R CNN
-F 2 "" H 1850 4250 50  0001 C CNN
+F 2 "Potentiometer_THT:Potentiometer_Bourns_PTV09A-1_Single_Vertical" H 1850 4250 50  0001 C CNN
 F 3 "~" H 1850 4250 50  0001 C CNN
 	1    1850 4250
@@
 F 0 "C11" H 1650 4750 50  0000 C CNN
 F 1 "0.1uF" H 1650 4850 50  0000 C CNN
-F 2 "" H 1888 4600 50  0001 C CNN
+F 2 "libraries:C_Flat_L7.2_H6.5" H 1888 4600 50  0001 C CNN
 F 3 "~" H 1850 4750 50  0001 C CNN
 	1    1850 4750
@@
 F 0 "RV2" H 2280 4096 50  0000 R CNN
 F 1 "Level" H 2280 4005 50  0000 R CNN
-F 2 "" H 2350 4050 50  0001 C CNN
+F 2 "Potentiometer_THT:Potentiometer_Bourns_PTV09A-1_Single_Vertical" H 2350 4050 50  0001 C CNN
 F 3 "~" H 2350 4050 50  0001 C CNN
 	1    2350 4050
@@
 F 0 "C12" V 3100 4050 50  0000 C CNN
 F 1 "0.047uF" V 3000 4050 50  0000 C CNN
-F 2 "" H 3288 3900 50  0001 C CNN
+F 2 "libraries:C_Flat_L7.2_H6.5" H 3288 3900 50  0001 C CNN
 F 3 "~" H 3250 4050 50  0001 C CNN
 	1    3250 4050
@@
 F 0 "C13" V 4600 4300 50  0000 C CNN
 F 1 "1uF" V 4500 4300 50  0000 C CNN
-F 2 "" H 4788 4150 50  0001 C CNN
+F 2 "libraries:C_Flat_L7.2_H10" H 4788 4150 50  0001 C CNN
 F 3 "~" H 4750 4300 50  0001 C CNN
 	1    4750 4300
@@
 F 0 "C15" H 7168 4646 50  0000 L CNN
 F 1 "100uF" H 7168 4555 50  0000 L CNN
-F 2 "" H 7088 4450 50  0001 C CNN
+F 2 "libraries:CP_Radial_D6.3mm_P2.00mm_L11.0mm" H 7088 4450 50  0001 C CNN
 F 3 "~" H 7050 4600 50  0001 C CNN
 	1    7050 4600
@@
 F 0 "C14" H 7968 4996 50  0000 L CNN
 F 1 "47uF" H 7968 4905 50  0000 L CNN
-F 2 "" H 7888 4800 50  0001 C CNN
+F 2 "libraries:CP_Radial_D6.3mm_P2.50mm_L7.0mm" H 7888 4800 50  0001 C CNN
 F 3 "~" H 7850 4950 50  0001 C CNN
 	1    7850 4950
