File: gndTest/gndTest.sch (KiCad schematic (older format))
At the start: 2 parts

Commit message: Minor changes
Connections:
- net InputJack renamed Amp
Changed lines of the file:
@@
 	4100 3750 4100 3650
 Text Label 4900 3950 2    50   ~ 0
-OutputJack
+Amp
 Wire Wire Line
 	4900 3950 4900 3500
