File: ConsolePedalUno/ConsolePedalUno.sch (KiCad schematic (older format))
At the start: 40 parts, among them J1 Conn_02x25_Counter_Clockwise, U1 TL972

Commit message: Working on new pedal
Parts:
- removed D1, D2: LED, LED_THT:LED_D5.0mm, symbol Device:LED
- removed R20: RLED, Resistor_THT:R_Axial_DIN0207_L6.3mm_D2.5mm_P10.16mm_Horizontal, symbol Device:R
- added C17: 100nF, libraries:C_Flat_L7.2_H6.5, symbol Device:C
- added D3, D4, D5, D6: LED, LED_THT:LED_D5.0mm, symbol Device:LED
- added J2: EXT, Connector_PinSocket_2.54mm:PinSocket_1x09_P2.54mm_Vertical, symbol Connector:Conn_01x09_Male
- added R14, R15, R16, R17: RLED, Resistor_THT:R_Axial_DIN0207_L6.3mm_D2.5mm_P10.16mm_Horizontal, symbol Device:R
- added R18, R19: 100K, Resistor_THT:R_Axial_DIN0207_L6.3mm_D2.5mm_P10.16mm_Horizontal, symbol Device:R
- added SW1, SW2, SW3, SW4: SW_Push, Button_Switch_THT:SW_PUSH_6mm, symbol Switch:SW_Push
- C1: value 0.1uF -> 100nF; footprint (none) -> libraries:C_Flat_L7.2_H6.5
- C10, C13: renamed from C?; footprint (none) -> libraries:CP_Radial_D5.0mm_P2.00mm_L11.0mm
- C11, C14, C5, C7, C8, C9: renamed from C?; footprint (none) -> libraries:C_Flat_L7.2_H6.5
- C12, C6: renamed from C?; footprint (none) -> Capacitor_THT:C_Axial_L3.8mm_D2.6mm_P7.50mm_Horizontal
- C15: renamed from C?; value 0.1uF -> 100nF; footprint (none) -> libraries:C_Flat_L7.2_H6.5
- C16: renamed from C?; footprint (none) -> libraries:CP_Radial_D6.3mm_P2.50mm_L7.0mm
- C2: footprint (none) -> libraries:C_Flat_L7.2_H6.5
- C3: footprint (none) -> libraries:CP_Radial_D5.0mm_P2.00mm_L11.0mm
- C4: footprint (none) -> Capacitor_THT:C_Axial_L3.8mm_D2.6mm_P7.50mm_Horizontal
- RV1: footprint (none) -> Potentiometer_THT:Potentiometer_Bourns_3386F_Vertical
- U1: footprint (none) -> Package_DIP:DIP-8_W7.62mm_Socket
- U3: renamed from U?; footprint Package_TO_SOT_THT:TO-220-3_Vertical -> Package_TO_SOT_THT:TO-220-3_Horizontal_TabDown
- Y1: renamed from Y?; footprint (none) -> Crystal:Crystal_HC49-U_Vertical
- gave numbers to parts that had none: 6
Connections:
- net +5V: now also J2.8 (Pin_8)
- net GND: now also D3.1 (K), D4.1 (K), D5.1 (K), D6.1 (K), J2.7 (Pin_7), R19.2, SW1.2, SW2.2, SW3.2, SW4.2
- net LEDPower: now also R18.1
- net pin1: now reaches R9.2, U2.1 (~RESET~/PC6)
- net pin1: now also C17.1, J2.9 (Pin_9)
- net DIG_5: now reaches U2.11 (PD5)
- net DIG_5: now also R15.1
- net DIG_6: now reaches U2.12 (PD6)
- net DIG_6: now also R16.1
- net DIG_11: now reaches U2.17 (PB3)
- net DIG_11: now also J2.6 (Pin_6), R17.1
- net DIG_12: now reaches U2.18 (PB4)
- net DIG_12: now also J2.5 (Pin_5), R18.2, R19.1
- net pin19: now reaches U2.19 (PB5)
- net pin19: now also J2.4 (Pin_4)
- net RX: now reaches U2.2 (PD0)
- net RX: now also J2.2 (Pin_2)
- net A2: now reaches U2.25 (PC2)
- net A2: now also SW1.1
- net A3: now reaches U2.26 (PC3)
- net A3: now also SW2.1
- net A4: now reaches U2.27 (PC4)
- net A4: now also SW3.1
- net A5: now reaches U2.28 (PC5)
- net A5: now also SW4.1
- net TX: now reaches U2.3 (PD1)
- net TX: now also J2.1 (Pin_1)
- net DIG_3: now reaches U2.5 (PD3)
- net DIG_3: now also R14.1
- new net: D3.2 (A), R14.2
- new net: D4.2 (A), R15.2
- new net: D5.2 (A), R16.2
- new net: D6.2 (A), R17.2
- new net: C17.2, J2.3 (Pin_3)
- no-connect marks 26 -> 33
