File: BadConnection/BadConnection.kicad_pcb (KiCad board)
At the start: 2 copper layers, 100 x 60 mm, 39 parts, among them J1 Conn_02x25_Counter_Clockwise, J2 Test Points, U1 TL072, U2 TL074, U3 CD4066BE

Commit message: Finalized and plotted board
Parts:
- C2, C5: moved to B.Cu
- moved R13 105.1 mm to (89.2, 105.7), turned to 90 degrees
- moved C7 85.3 mm to (170.6, 88.5), turned to 180 degrees
- moved R3 83.7 mm to (176.4, 95.5), turned to 270 degrees
- moved C3 73.8 mm to (135.2, 93.6), turned to 180 degrees
- moved R11 71.4 mm to (161.4, 107.8), turned to 180 degrees
- moved R1 71.0 mm to (140.7, 104.1), turned to 90 degrees
- moved C1 69.3 mm to (109.2, 104.3), turned to 180 degrees
- moved D1 68.5 mm to (117.2, 101.1), turned to 270 degrees
- moved C4 66.4 mm to (97.3, 88.5), turned to 180 degrees
- moved D2 62.4 mm to (85.2, 90.3), turned to 90 degrees
- moved R12 62.4 mm to (104.3, 111.3)
- moved C6 61.4 mm to (161.4, 104.1), turned to 180 degrees
- moved R6 61.2 mm to (106.4, 77.5), turned to 270 degrees
- moved R8 59.5 mm to (90.8, 74.0)
- moved R2 57.3 mm to (144.7, 94.0), turned to 270 degrees
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Routing:
- net /pin13: track 0.00 -> 144.8 mm, vias 0 -> 1
- net +9V: track 61.6 -> 205.7 mm, vias 2 -> 4
- net /VREF: track 0.00 -> 123.1 mm
- net /pin1: track 0.00 -> 105.5 mm, vias 0 -> 2
- net /M2: track 0.00 -> 96.3 mm, vias 0 -> 1
- net Net-(C5-Pad2): track 0.00 -> 87.3 mm, vias 0 -> 1
- net /Output: track 0.00 -> 86.1 mm, vias 0 -> 2
- net Net-(RV1-Pad2): track 0.00 -> 54.5 mm, vias 0 -> 1
- net /LEDPower: track 55.9 -> 110.0 mm, vias 2 -> 4
- net Net-(R14-Pad1): track 0.00 -> 50.0 mm, vias 0 -> 1
- net /M1: track 0.00 -> 46.7 mm
- net Net-(C1-Pad1): track 0.00 -> 41.7 mm
- net Net-(D1-Pad2): track 0.00 -> 41.5 mm, vias 0 -> 1
- net /pin2: track 0.00 -> 38.0 mm, vias 0 -> 1
- net /Input: track 126.0 -> 90.7 mm, vias 4 -> 2
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