File: GuitarMicroBoard/GuitarMicroBoard.kicad_pcb (KiCad board)
At the start: 2 copper layers, 66 x 29.5 mm, 24 parts, among them J1 Power, J2 OLED Power, J3 OLED I2C, J4 Input, U1 ATmega328P-PU, U2 TL972, U3 L78L33_TO92

Commit message: Finalized microcontroller guitar board
Parts:
- moved C1 57.1 mm to (163.4, 112.8), turned to 270 degrees
- moved C2 49.1 mm to (131.1, 117.3)
- moved C4 44.2 mm to (128.0, 117.3), turned to 180 degrees
- moved C5 35.6 mm to (148.3, 92.1), turned to 0 degrees
- moved R2 29.6 mm to (166.8, 92.1), turned to 180 degrees
- moved R3 29.2 mm to (138.9, 117.3)
- moved R8 25.3 mm to (122.7, 92.1)
- moved R7 25.3 mm to (135.4, 92.1)
- moved U3 23.4 mm to (178.7, 93.1)
- moved R6 17.7 mm to (167.0, 95.1)
- moved C7 16.5 mm to (181.1, 97.0), turned to 270 degrees
- moved R4 13.8 mm to (150.9, 105.7)
- moved R1 13.7 mm to (167.0, 118.1)
- moved R5 12.9 mm to (161.0, 109.1), turned to 180 degrees
- moved C6 8.46 mm to (173.7, 101.9), turned to 180 degrees
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Routing:
- net +3V3: track 0.00 -> 74.8 mm
- net /VREF: track 0.00 -> 73.7 mm, vias 0 -> 1
- net Net-(C1-Pad1): track 0.00 -> 52.8 mm, vias 0 -> 2
- net Net-(C4-Pad2): track 0.00 -> 50.6 mm
- net Net-(C4-Pad1): track 0.00 -> 30.0 mm
- net /A0: track 0.00 -> 26.4 mm
- net +9V: track 0.00 -> 25.7 mm
- net /Guitar: track 0.00 -> 14.7 mm
- net Net-(C3-Pad1): track 0.00 -> 14.5 mm
- net /ButtonB: track 0.00 -> 12.9 mm
- net /SDA: track 0.00 -> 11.2 mm
- net Net-(R4-Pad1): track 0.00 -> 9.93 mm
- net GND: track 0.00 -> 6.87 mm, vias 0 -> 3
- net Net-(C2-Pad2): track 0.00 -> 6.74 mm
- net /SCL: track 0.00 -> 6.53 mm
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- added copper zone on B.Cu, net GND
- added copper zone on F.Cu, net GND
Other:
- board text added: "3.3V"
- board text added: "9V"
- board text added: "Button"
- board text added: "GND"
- board text added: "Guitar"
- board text added: "JLCJLCJLCJLC"
- board text added: "SCL"
- board text added: "SDA"
- board text added: "Thomas McDonagh consolepedals.com Guitar Micro Board V1.0"
