File: InternalAmpLM386/InternalAmpLM386.kicad_pcb (KiCad board)
At the start: 2 copper layers, 78 x 58.5 mm, 23 parts, among them J1 Conn_01x04_Male, J2 Speaker, J3 Power, Q1 MPF102, SW1 Power, U1 LM386

Commit message: Finalized speaker board
Parts:
- removed H3, H4: Mount, MountingHole:MountingHole_2.7mm_Pad
- C2, C3, C4, RV2: moved to B.Cu
- moved J1 130.6 mm to (166.9, 93.5), turned to 180 degrees
- moved R1 129.6 mm to (156.2, 111.3)
- moved R2 119.2 mm to (156.2, 114.6)
- moved C4 115.5 mm to (158.8, 117.3)
- moved H2 104.7 mm to (156.8, 125.8)
- moved C3 104.0 mm to (157.5, 93.7), turned to 180 degrees
- moved R3 98.0 mm to (124.7, 107.7)
- moved C2 89.3 mm to (99.3, 111.5), turned to 180 degrees
- moved C5 88.7 mm to (119.4, 117.3), turned to 90 degrees
- moved RV2 87.0 mm to (132.5, 112.3), turned to 270 degrees
- moved Q1 86.2 mm to (160.0, 106.4)
- moved C1 84.7 mm to (139.7, 113.8), turned to 270 degrees
- moved J3 82.5 mm to (157.5, 82.0), turned to 270 degrees
- moved R4 81.8 mm to (105.7, 114.8), turned to 90 degrees
- moved D1 74.8 mm to (97.0, 99.8), turned to 90 degrees
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Routing:
- net Net-(C1-Pad1): track 0.00 -> 97.2 mm, vias 0 -> 1
- net 9V: track 0.00 -> 91.8 mm
- net Net-(C2-Pad1): track 0.00 -> 87.8 mm
- net Net-(C3-Pad2): track 0.00 -> 52.3 mm, vias 0 -> 1
- net Net-(C5-Pad2): track 0.00 -> 50.2 mm, vias 0 -> 1
- net Net-(RV2-Pad2): track 0.00 -> 42.5 mm
- net Net-(RV2-Pad1): track 0.00 -> 35.4 mm
- net Net-(C5-Pad1): track 0.00 -> 33.9 mm
- net Net-(D2-Pad1): track 0.00 -> 32.9 mm, vias 0 -> 1
- net Input: track 0.00 -> 31.1 mm
- net Net-(C4-Pad1): track 0.00 -> 28.0 mm
- net Net-(C2-Pad2): track 0.00 -> 16.3 mm
- net Net-(D1-Pad2): track 0.00 -> 13.2 mm
- net Net-(RV1-Pad2): track 0.00 -> 8.58 mm
- added copper zone on B.Cu, net GND
- added copper zone on F.Cu, net GND
Other:
- board size 78 x 58.5 mm -> 78 x 50.5 mm
- board text added: "9V"
- board text added: "GND"
- board text added: "In"
- board text added: "JLCJLCJLCJLC"
- board text added: "Thomas McDonagh consolepedals.com Internal LM386 Amp V1.0"
