File: FmReceiverCartridge/FmReceiverCartridge.kicad_pcb (KiCad board)
At the start: 2 copper layers, 100 x 60 mm, 33 parts, among them J1 Jumper, J2 Conn_02x25_Counter_Clockwise, Q1 2N3904, SW1 SW_A, SW2 SW_B, U1 ATtiny84A-PU, U2 ISD1820P, U3 L78L05_TO92

Commit message: Finalized and exported fm receiver board
Parts:
- removed C2: 100uF, libraries:CP_Radial_D6.3mm_P2.50mm
- removed C3: 220uF, libraries:CP_Radial_D6.3mm_P2.50mm
- removed D3: LED, Connector_PinSocket_2.54mm:PinSocket_1x02_P2.54mm_Vertical
- removed J1: Jumper, Connector_PinSocket_2.54mm:PinSocket_1x02_P2.54mm_Vertical
- removed Q1: 2N3904, Package_TO_SOT_THT:TO-92_Inline
- removed R10: 100K, Resistor_THT:R_Axial_DIN0207_L6.3mm_D2.5mm_P10.16mm_Horizontal
- removed R3: 47K, Resistor_THT:R_Axial_DIN0207_L6.3mm_D2.5mm_P10.16mm_Horizontal
- removed R6, R7, R8: 1K, Resistor_THT:R_Axial_DIN0207_L6.3mm_D2.5mm_P10.16mm_Horizontal
- removed R9: RLED, Resistor_THT:R_Axial_DIN0207_L6.3mm_D2.5mm_P10.16mm_Horizontal
- C1: value 0.1uF -> 1uF; footprint libraries:C_Flat_L7.2_H6.5 -> libraries:C_Flat_L7.2_H10
- R1: value 47K -> 100R
- R2: value 1K -> 100R
- RV1: value 500KL Volume -> 500K
- SW1, SW2: footprint Button_Switch_THT:SW_PUSH_6mm -> TL2230EEF140-LatchSwitch:TL2230OAF140
- U1: value ATtiny84A-PU -> ATmega328P-PU; footprint Package_DIP:DIP-14_W7.62mm -> Package_DIP:DIP-28_W7.62mm
- U2: value ISD1820P -> Si470xBreakout; footprint Package_DIP:DIP-14_W7.62mm -> libraries:Si470xBreakout
- U3: value L78L05_TO92 -> L78L33_TO92
- moved C4 52.5 mm to (92.5, 84.3)
- moved R2 44.6 mm to (120.1, 90.9)
- moved R1 38.5 mm to (135.2, 90.9), turned to 0 degrees
- moved C1 30.5 mm to (98.0, 99.1), turned to 0 degrees
- moved U1 27.5 mm to (116.2, 108.7), turned to 90 degrees
- moved U3 12.6 mm to (101.8, 92.5), turned to 180 degrees
- moved U2 11.6 mm to (172.7, 90.9)
- moved R12 9.96 mm to (155.2, 91.2)
- moved R5 9.96 mm to (155.2, 88.9)
- moved R11 9.89 mm to (110.2, 101.3)
- moved R4 9.89 mm to (110.2, 88.9)
- moved SW1 4.91 mm to (98.5, 83.8)
- moved SW2 4.91 mm to (163.0, 83.8)
- moved C5 3.09 mm to (92.5, 107.7)
Connections:
- C1 pad 1: Net-(C1-Pad1) -> /Output
- C1 pad 2: Net-(C1-Pad2) -> /Input
- C5 pad 2: +5V -> +3V3
- J2 pad 22: /Input -> /Output
- J2 pad 29: /Input -> /Output
- J2 pad 4: /Input -> /Output
- J2 pad 47: /Input -> /Output
- R1 pad 2: /Input -> Net-(R1-Pad2)
- R2 pad 1: GND -> Net-(R2-Pad1)
- RV1 pad 1: Net-(R7-Pad1) -> Net-(R1-Pad1)
- RV1 pad 2: /Input -> /Output
- SW1 pad 1: /SW_A -> (no net)
- SW1 pad 2: GND -> /SW_A
- SW2 pad 1: /SW_B -> (no net)
- SW2 pad 2: GND -> /SW_B
- U1 pad 1: +5V -> (no net)
- U1 pad 10: /PLAYL -> (no net)
- U1 pad 11: /PLAYE -> (no net)
- U1 pad 12: /REC -> /LED_A
- U1 pad 14: GND -> (no net)
- U1 pad 2: /SW_A -> (no net)
- U1 pad 3: /SW_B -> (no net)
- U1 pad 4: (no net) -> /D2
- U1 pad 5: /LED_B -> /D3
- U1 pad 7: /Loop -> +3V3
- U1 pad 8: /LED_A -> GND
- U1 pad 9: /FT -> (no net)
- U2 pad 1: /REC -> Net-(R1-Pad2)
- U2 pad 10: Net-(J1-Pad1) -> /D3
- U2 pad 2: /PLAYE -> Net-(R2-Pad1)
- U2 pad 3: /PLAYL -> GND
- U2 pad 4: Net-(C1-Pad2) -> +3V3
- U2 pad 5: (no net) -> /SDA
- U2 pad 6: (no net) -> /SCL
- U2 pad 7: GND -> (no net)
- U2 pad 8: GND -> /D2
- U2 pad 9: Net-(C2-Pad1) -> (no net)
- U3 pad 1: +5V -> +3V3
Routing:
- net +3V3: track 0.00 -> 187.5 mm, vias 0 -> 1
- net +5V: track 172.1 -> 0.00 mm, vias 1 -> 0
- net /Output: track 0.00 -> 149.0 mm, vias 0 -> 4
- net /Input: track 225.3 -> 97.1 mm, vias 5 -> 2
- net /FT: track 104.0 -> 0.00 mm, vias 1 -> 0
- net /PLAYE: track 98.6 -> 0.00 mm, vias 1 -> 0
- net Net-(R2-Pad1): track 0.00 -> 71.7 mm
- net /PLAYL: track 71.5 -> 0.00 mm, vias 2 -> 0
- net /SCL: track 0.00 -> 63.9 mm, vias 0 -> 1
- net /REC: track 62.3 -> 0.00 mm, vias 1 -> 0
- net /SW_B: track 85.2 -> 28.5 mm, vias 1 -> 0
- net /SDA: track 0.00 -> 56.5 mm, vias 0 -> 1
- net /D2: track 0.00 -> 51.4 mm, vias 0 -> 1
- net /D3: track 0.00 -> 50.2 mm, vias 0 -> 1
- net Net-(C1-Pad2): track 50.0 -> 0.00 mm, vias 1 -> 0
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Other:
- board text added: "FM Receiver V1.0"
- board text removed: "Chip Loop V1.1"
- board text removed: "Play"
- board text removed: "Record"
- board text removed: "Volume"
