File: FmTransmitterCartridge/FmTransmitterCartridge.sch (KiCad schematic (older format))
At the start: 21 parts, among them J2 Conn_02x25_Counter_Clockwise, SW1 SW_A, SW2 SW_B, U1 ATmega328P-PU

Commit message: Finalized schematic
Parts:
- added C10: 1uF, libraries:C_Flat_L7.2_H10, symbol Device:C
- added C2, C9: 4.7uF, libraries:CP_Radial_D5.0mm_P2.00mm_L11.0mm, symbol Device:CP
- added C6, C8: 6.8nF, libraries:C_Flat_L7.2_H6.5, symbol Device:C
- added C7: 270pF, libraries:C_Flat_L7.2_H6.5, symbol Device:C
- added R10, R7, R9: 100K, Resistor_THT:R_Axial_DIN0207_L6.3mm_D2.5mm_P10.16mm_Horizontal, symbol Device:R
- added R2, R6, R8: 4.7K, Resistor_THT:R_Axial_DIN0207_L6.3mm_D2.5mm_P10.16mm_Horizontal, symbol Device:R
- added R3: 1M, Resistor_THT:R_Axial_DIN0207_L6.3mm_D2.5mm_P10.16mm_Horizontal, symbol Device:R
- added RV1: 500K, Potentiometer_THT:Potentiometer_Bourns_3386F_Vertical, symbol Device:R_POT
- added U3: TL972, Package_DIP:DIP-8_W7.62mm, symbol Device:Opamp_Dual_Generic
- C3: renamed from C?; footprint libraries:C_Flat_L7.2_H10 -> libraries:C_Flat_L7.2_H6.5
- U2: renamed from U?; footprint (none) -> libraries:Si4713Breakout
- gave numbers to parts that had none: 2
Connections:
- net +5V: now also U2.3 (VIN), R9.1, U3.8 (V+)
- net GND: now also R1.1, U2.4 (GND), C2.2, C6.1, C8.1, C9.2, R10.2, U3.4 (V-)
- net Input: now also C3.2, R1.2
- net SCL: now also U2.9 (SCL)
- net SDA: now also U2.8 (SDA)
- net D12: now reaches U1.18 (PB4)
- net D12: now also U2.11 (RST)
- net at U2.1 (LIN): now also U2.2 (RIN), C10.2
- net at C3.1: now also R3.2, R6.1
- new net: C6.2, R6.2, U3.5 (+)
- new net: U3.1, U3.2 (-)
- new net: C7.2, R7.1, RV1.1, RV1.2, U3.6 (-)
- new net: C7.1, R7.2, R8.1, U3.7
- new net: R2.2, RV1.3
- new net: C2.1, R2.1
- new net PreAmp: C10.1, C8.2, R8.2
- new net VREF: C9.1, R10.1, R3.1, R9.2, U3.3 (+)
- no-connect marks 44 -> 47
Other:
- moved on the sheet: C1, U2
