File: FmTransmitterCartridge/FmTransmitterCartridge.kicad_pcb (KiCad board)
At the start: 2 copper layers, 100 x 60 mm, 36 parts, among them J2 Conn_02x25_Counter_Clockwise, SW1 SW_A, SW2 SW_B, U1 ATmega328P-PU, U2 Si4713Breakout, U3 TL972, U4 L78L05_TO92

Commit message: Finalized FM Transmitter cartridge
Routing:
- net /PreAmp: track 10.3 -> 55.9 mm, vias 0 -> 1
- net Net-(C10-Pad2): track 2.54 -> 43.4 mm, vias 0 -> 1
