File: ChipLoop/ChipLoop.sch (KiCad schematic (older format))
At the start: 17 parts, among them J1 Conn_02x25_Counter_Clockwise, Q1 2N3904

Commit message: Minor changes
Parts:
- added R?: 4.7K, Resistor_THT:R_Axial_DIN0207_L6.3mm_D2.5mm_P10.16mm_Horizontal, symbol Device:R
- added U?: ISD1820P, symbol ISD1820P:ISD1820P
Other:
- moved on the sheet: C?
Changed lines of the file:
@@
 	10000 5250 10000 5350
 Connection ~ 10000 5350
-Text Label 4150 3700 2    50   ~ 0
+Text Label 2700 4250 2    50   ~ 0
 Input
 $Comp
 L Device:C C?
 U 1 1 6172FFFD
-P 4700 3650
-F 0 "C?" V 4550 3600 50  0000 L CNN
-F 1 "0.1uF" V 4850 3550 50  0000 L CNN
-F 2 "libraries:C_Flat_L7.2_H6.5" H 4738 3500 50  0001 C CNN
-F 3 "~" H 4700 3650 50  0001 C CNN
-	1    4700 3650
+P 3150 4000
+F 0 "C?" V 3000 3950 50  0000 L CNN
+F 1 "0.1uF" V 3300 3900 50  0000 L CNN
+F 2 "libraries:C_Flat_L7.2_H6.5" H 3188 3850 50  0001 C CNN
+F 3 "~" H 3150 4000 50  0001 C CNN
+	1    3150 4000
 	0    1    1    0
 $EndComp
+$Comp
+L ISD1820P:ISD1820P U?
+U 1 1 6173B7F0
+P 5150 4450
+F 0 "U?" H 5150 4975 50  0000 C CNN
+F 1 "ISD1820P" H 5150 4884 50  0000 C CNN
+F 2 "" H 5150 4450 50  0001 C CNN
+F 3 "" H 5150 4450 50  0001 C CNN
+	1    5150 4450
+	1    0    0    -1
+$EndComp
+$Comp
+L Device:R R?
+U 1 1 6173D6F3
+P 3050 3550
+F 0 "R?" V 2950 3500 50  0000 L CNN
+F 1 "4.7K" V 3150 3450 50  0000 L CNN
+F 2 "Resistor_THT:R_Axial_DIN0207_L6.3mm_D2.5mm_P10.16mm_Horizontal" V 2980 3550 50  0001 C CNN
+F 3 "~" H 3050 3550 50  0001 C CNN
+	1    3050 3550
+	0    1    1    0
+$EndComp

Commit message: Minor changes
Parts:
- added C2: 0.1uF, libraries:C_Flat_L7.2_H6.5, symbol Device:C
- added R?: 4.7K, Resistor_THT:R_Axial_DIN0207_L6.3mm_D2.5mm_P10.16mm_Horizontal, symbol Device:R
- gave numbers to parts that had none: 1
Connections:
- net GND: now also C1.2
- net Input: now also C2.2
- net at C1.1: now also U?.5 (MICREF)
- net at U?.4 (MIC): now also C2.1
Other:
- moved on the sheet: C1, U?
Changed lines of the file:
@@
 	10000 5250 10000 5350
 Connection ~ 10000 5350
-Text Label 2700 4250 2    50   ~ 0
+Text Label 2700 4450 2    50   ~ 0
 Input
 $Comp
-L Device:C C?
+L Device:C C1
 U 1 1 6172FFFD
-P 3150 4000
-F 0 "C?" V 3000 3950 50  0000 L CNN
-F 1 "0.1uF" V 3300 3900 50  0000 L CNN
-F 2 "libraries:C_Flat_L7.2_H6.5" H 3188 3850 50  0001 C CNN
-F 3 "~" H 3150 4000 50  0001 C CNN
-	1    3150 4000
+P 3100 4850
+F 0 "C1" V 2950 4800 50  0000 L CNN
+F 1 "0.1uF" V 3250 4750 50  0000 L CNN
+F 2 "libraries:C_Flat_L7.2_H6.5" H 3138 4700 50  0001 C CNN
+F 3 "~" H 3100 4850 50  0001 C CNN
+	1    3100 4850
 	0    1    1    0
 $EndComp
@@
 L ISD1820P:ISD1820P U?
 U 1 1 6173B7F0
-P 5150 4450
-F 0 "U?" H 5150 4975 50  0000 C CNN
-F 1 "ISD1820P" H 5150 4884 50  0000 C CNN
-F 2 "" H 5150 4450 50  0001 C CNN
-F 3 "" H 5150 4450 50  0001 C CNN
-	1    5150 4450
+P 5750 4500
+F 0 "U?" H 5750 5025 50  0000 C CNN
+F 1 "ISD1820P" H 5750 4934 50  0000 C CNN
+F 2 "" H 5750 4500 50  0001 C CNN
+F 3 "" H 5750 4500 50  0001 C CNN
+	1    5750 4500
 	1    0    0    -1
 $EndComp
@@
 	0    1    1    0
 $EndComp
+$Comp
+L power:GND #PWR?
+U 1 1 617C339E
+P 2700 4650
+F 0 "#PWR?" H 2700 4400 50  0001 C CNN
+F 1 "GND" H 2600 4650 50  0000 C CNN
+F 2 "" H 2700 4650 50  0001 C CNN
+F 3 "" H 2700 4650 50  0001 C CNN
+	1    2700 4650
+	1    0    0    -1
+$EndComp
+$Comp
+L Device:C C2
+U 1 1 617C49B2
+P 3100 4250
+F 0 "C2" V 2950 4200 50  0000 L CNN
+F 1 "0.1uF" V 3250 4150 50  0000 L CNN
+F 2 "libraries:C_Flat_L7.2_H6.5" H 3138 4100 50  0001 C CNN
+F 3 "~" H 3100 4250 50  0001 C CNN
+	1    3100 4250
+	0    1    1    0
+$EndComp
+Wire Wire Line
+	2700 4450 2850 4450
+Wire Wire Line
+	2850 4450 2850 4250
+Wire Wire Line
+	2850 4250 2950 4250
+Wire Wire Line
+	2700 4650 2850 4650
+Wire Wire Line
+	2850 4650 2850 4850
+Wire Wire Line
+	2850 4850 2950 4850
+$Comp
+L Device:R R?
+U 1 1 617C9ABC
+P 3100 5500
+F 0 "R?" V 3000 5450 50  0000 L CNN
+F 1 "4.7K" V 3200 5400 50  0000 L CNN
+F 2 "Resistor_THT:R_Axial_DIN0207_L6.3mm_D2.5mm_P10.16mm_Horizontal" V 3030 5500 50  0001 C CNN
+F 3 "~" H 3100 5500 50  0001 C CNN
+	1    3100 5500
+	0    1    1    0
+$EndComp
+Wire Wire Line
+	3250 4250 3350 4250
+Wire Wire Line
+	3350 4250 3350 4500
+Wire Wire Line
+	3350 4500 5250 4500
+Wire Wire Line
+	5250 4600 3350 4600
+Wire Wire Line
+	3350 4600 3350 4850
+Wire Wire Line
+	3350 4850 3250 4850
 $EndSCHEMATC

Commit message: Still trying to figure out what I need to change
Parts:
- removed C1, C2: 0.1uF, libraries:C_Flat_L7.2_H6.5, symbol Device:C
- removed D3, D4: 1N4148, Diode_THT:D_DO-35_SOD27_P7.62mm_Horizontal, symbol Diode:1N4148
- removed Q1: 2N3904, Package_TO_SOT_THT:TO-92_Inline, symbol Transistor_BJT:2N3904
- removed R1: 2M, Resistor_THT:R_Axial_DIN0207_L6.3mm_D2.5mm_P10.16mm_Horizontal, symbol Device:R
- removed R2: 4.7K, Resistor_THT:R_Axial_DIN0207_L6.3mm_D2.5mm_P10.16mm_Horizontal, symbol Device:R
- removed RV1: 250K Distortion, Potentiometer_THT:Potentiometer_Bourns_PTV09A-1_Single_Vertical, symbol Device:R_POT
- removed RV2: 250K Volume, Potentiometer_THT:Potentiometer_Bourns_PTV09A-1_Single_Vertical, symbol Device:R_POT
- added C?: 0.001uF, libraries:C_Flat_L7.2_H6.5, symbol Device:C
- added C?: 4.7uF, symbol Device:CP
- added C? (x2): 0.1uF, libraries:C_Flat_L7.2_H6.5, symbol Device:C
- added C?: 0.33uF, libraries:C_Flat_L7.2_H6.5, symbol Device:C
- added D?: LED, LED_THT:LED_D5.0mm, symbol Device:LED
- added R?: RLED, Resistor_THT:R_Axial_DIN0207_L6.3mm_D2.5mm_P10.16mm_Horizontal, symbol Device:R
- added SW? (x3): SW, symbol Switch:SW_Push
- added SW? (x2): SW_SPDT, symbol Switch:SW_SPDT
- added U?: ATtiny84A-PU, Package_DIP:DIP-14_W7.62mm, symbol MCU_Microchip_ATtiny:ATtiny84A-PU
- added U?: LM7805_TO220, Package_TO_SOT_THT:TO-220-3_Vertical, symbol Regulator_Linear:LM7805_TO220
Connections:
- net +9V: now also C?.2, U?.1 (VI)
- net GND: now also R?.1, R?.2, U?.14 (VSSD), U?.7 (SP-), U?.8 (VSSA), C?.1, C?.1, C?.1, C?.1, C?.2, U?.14 (GND), U?.2 (GND)
- net Output: now also U?.9 (SP+)
- net at U?.1 (REC): now also C?.2, SW?.2
- net at U?.11 (VCC): now also C?.2, R?.2
- net at U?.13 (RECLED): now also D?.1 (K), SW?.1 (A)
- net at U?.2 (PLAYE): now also SW?.2, SW?.2 (B)
- net at U?.3 (PLAYL): now also SW?.2
- net at U?.6 (AGC): now also C?.1
- new net: SW?.1, SW?.1, SW?.1
- new net: D?.2 (A), R?.1
- new net +5V: C?.2, U?.3 (VO)
Other:
- moved on the sheet: R?

Commit message: Finalized project
Parts:
- removed R?: 4.7K, Resistor_THT:R_Axial_DIN0207_L6.3mm_D2.5mm_P10.16mm_Horizontal, symbol Device:R
- removed SW? (x3): SW, symbol Switch:SW_Push
- removed SW? (x2): SW_SPDT, symbol Switch:SW_SPDT
- removed U?: LM7805_TO220, Package_TO_SOT_THT:TO-220-3_Vertical, symbol Regulator_Linear:LM7805_TO220
- added C4: 220uF, libraries:CP_Radial_D6.3mm_P2.50mm, symbol Device:CP
- added D2, D3: LED, LED_THT:LED_D5.0mm, symbol Device:LED
- added J2: Jumper, Connector_PinSocket_2.54mm:PinSocket_1x02_P2.54mm_Vertical, symbol Connector:Conn_01x02_Male
- added Q1: 2N3904, Package_TO_SOT_THT:TO-92_Inline, symbol Transistor_BJT:2N3904
- added R1, R8: 1K, Resistor_THT:R_Axial_DIN0207_L6.3mm_D2.5mm_P10.16mm_Horizontal, symbol Device:R
- added R4: 100K, Resistor_THT:R_Axial_DIN0207_L6.3mm_D2.5mm_P10.16mm_Horizontal, symbol Device:R
- added R6, R7: RLED, Resistor_THT:R_Axial_DIN0207_L6.3mm_D2.5mm_P10.16mm_Horizontal, symbol Device:R
- added RV1: 500KL Volume, Potentiometer_THT:Potentiometer_Bourns_PTV09A-1_Single_Vertical, symbol Device:R_POT
- added SW1: SW_A, Button_Switch_THT:SW_PUSH_6mm, symbol Switch:SW_Push
- added SW2: SW_B, Button_Switch_THT:SW_PUSH_6mm, symbol Switch:SW_Push
- added U3: L78L05_TO92, Package_TO_SOT_THT:TO-92_Inline, symbol Regulator_Linear:L78L05_TO92
- C5: renamed from C?; footprint (none) -> libraries:CP_Radial_D5.0mm_P2.00mm
- D1: renamed from D?; footprint LED_THT:LED_D5.0mm -> Connector_PinSocket_2.54mm:PinSocket_1x02_P2.54mm_Vertical
- U2: renamed from U?; footprint (none) -> Package_DIP:DIP-14_W7.62mm
- gave numbers to parts that had none: 11
- renumbered C1 to C3
Connections:
- net +5V: now also C1.2, R5.2, U1.1 (VCC), U2.11 (VCC), R1.2, U3.1 (VO)
- net +9V: now also U3.3 (VI)
- net GND: now also C4.2, D2.1 (K), D3.1 (K), R4.2, RV1.3, SW1.2, SW2.2, U3.2 (GND)
- net Input: now also J1.22 (Pin_22), J1.29 (Pin_29), J1.4 (Pin_4), J1.47 (Pin_47), R2.2, RV1.2
- net REC: now reaches C6.2, U2.1 (REC)
- net REC: now also U1.12 (PA1)
- net at U2.10 (ROSC): now also J2.1 (Pin_1)
- net FT: now reaches U2.12 (FT)
- net FT: now also U1.9 (PA4)
- net at D1.1 (K), U2.13 (RECLED): now also Q1.3 (C)
- net PLAYE: now reaches U2.2 (PLAYE)
- net PLAYE: now also U1.11 (PA2), Q1.1 (E)
- net PLAYL: now reaches U2.3 (PLAYL)
- net PLAYL: now also U1.10 (PA3)
- net at R2.1: now also C4.1, R1.1
- net SW_A: now reaches U1.2 (XTAL1/PB0)
- net SW_A: now also SW1.1
- net SW_B: now reaches U1.3 (XTAL2/PB1)
- net SW_B: now also SW2.1
- net LED_B: now reaches U1.5 (PB2)
- net LED_B: now also R7.1
- net Loop: now reaches U1.7 (PA6)
- net Loop: now also R8.2
- net LED_A: now reaches U1.8 (PA5)
- net LED_A: now also R6.1
- removed net Output: J1.22 (Pin_22), J1.29 (Pin_29), J1.4 (Pin_4), J1.47 (Pin_47), U2.9 (SP+)
- new net: RV1.1, U2.9 (SP+)
- new net: Q1.2 (B), R8.1
- new net: J2.2 (Pin_2), R4.1
- new net: D2.2 (A), R6.2
- new net: D3.2 (A), R7.2
- no-connect marks 26 -> 29
Other:
- moved on the sheet: C1, C2, C3, C5, C6, D1, R2, R5, U2

Commit message: Finalized changes to chip loop input and output
Parts:
- removed C2, C3: 0.1uF, libraries:C_Flat_L7.2_H6.5, symbol Device:C
- removed C5: 4.7uF, libraries:CP_Radial_D5.0mm_P2.00mm, symbol Device:CP
- removed C6: 0.001uF, libraries:C_Flat_L7.2_H6.5, symbol Device:C
- added C2: 100uF, libraries:CP_Radial_D6.3mm_P2.50mm, symbol Device:CP
- added R1, R3: 47K, Resistor_THT:R_Axial_DIN0207_L6.3mm_D2.5mm_P10.16mm_Horizontal, symbol Device:R
- added R7: 1K, Resistor_THT:R_Axial_DIN0207_L6.3mm_D2.5mm_P10.16mm_Horizontal, symbol Device:R
- R2: value 4.7K -> 1K
- renumbered C4 to C3, C7 to C4, C8 to C5, D2 to D1, D3 to D2, D1 to D3, J2 to J1, J1 to J2, R4 to R10, R9 to R11, R10 to R12, R6 to R4, R7 to R5, R8 to R6, R1 to R8, R5 to R9
Connections:
- net +5V: no longer C1.2
- net GND: now also R2.1; no longer C1.1, U2.14 (VSSD)
- net Input: now also R1.2; no longer R2.2
- net at U2.4 (MIC): now also C1.2
- net at U2.9 (SP+): now also C2.1; no longer RV1.1
- net at C3.1, R8.1: no longer R2.1
- new net: R7.1, RV1.1
- new net: R1.1, R2.2, R3.2
- new net: C1.1, R3.1
- new net: C2.2, R7.2
Other:
- moved on the sheet: RV1
