File: ConsolePedalSide/ConsolePedalSide.sch (KiCad schematic (older format))
At the start: 16 parts, among them J1 AudioJack3, J2 AudioJack2, J3 SlotA, J4 SlotB

Commit message: Made pin holes wider for easier hand soldering
Parts:
- J1: footprint Connector_PinSocket_2.54mm:PinSocket_1x03_P2.54mm_Vertical -> libraries:Pins_1x03_Wide
- J2: footprint Connector_PinSocket_2.54mm:PinSocket_1x02_P2.54mm_Vertical -> libraries:Pins_1x02_Wide
Changed lines of the file:
@@
 F 0 "J1" H 1282 2175 50  0000 C CNN
 F 1 "AudioJack3" H 1282 2084 50  0000 C CNN
-F 2 "Connector_PinSocket_2.54mm:PinSocket_1x03_P2.54mm_Vertical" H 1300 1850 50  0001 C CNN
+F 2 "libraries:Pins_1x03_Wide" H 1300 1850 50  0001 C CNN
 F 3 "" H 1300 1850 50  0001 C CNN
 	1    1300 1850
@@
 F 0 "J2" H 6032 2275 50  0000 C CNN
 F 1 "AudioJack2" H 6032 2184 50  0000 C CNN
-F 2 "Connector_PinSocket_2.54mm:PinSocket_1x02_P2.54mm_Vertical" H 6000 1950 50  0001 C CNN
+F 2 "libraries:Pins_1x02_Wide" H 6000 1950 50  0001 C CNN
 F 3 "" H 6000 1950 50  0001 C CNN
 	1    6000 1950
