File: ConsolePedal8BitarSMT/ConsolePedal8BitarSMT.sch (KiCad schematic (older format))
At the start: 27 parts, among them IC1 CD4069UBE, J1 Conn_02x25_Counter_Clockwise, Q1 2N3904

Commit message: Finalized SMT project and fixed minor issues
Parts:
- removed D3: 1N4001, Diode_THT:D_DO-41_SOD81_P10.16mm_Horizontal, symbol Diode:1N4001
- removed Q1: 2N3904, Package_TO_SOT_THT:TO-92_Inline, symbol Transistor_BJT:2N3904
- added IC2: CD4069UBM, Package_SO:SOIC-14_3.9x8.7mm_P1.27mm, symbol SamacSys_Parts:CD4069UBE
- added Q1: MMBT3904, Package_TO_SOT_SMD:SOT-23, symbol Transistor_BJT:MMBT3904
- added R11: RLED, Resistor_THT:R_Axial_DIN0207_L6.3mm_D2.5mm_P10.16mm_Horizontal, symbol Device:R
- added R12, R13: 22K, Resistor_SMD:R_0603_1608Metric, symbol Device:R
- C1, C3: footprint libraries:C_Flat_L7.2_H6.5 -> Capacitor_SMD:C_0603_1608Metric; LCSC (none) -> C14663
- C2: footprint libraries:C_Flat_L7.2_H6.5 -> Capacitor_SMD:C_0603_1608Metric; LCSC (none) -> C1604
- C4: footprint libraries:C_Flat_L7.2_H6.5 -> Capacitor_SMD:C_0603_1608Metric; LCSC (none) -> C53987
- C5, C8: footprint Capacitor_THT:CP_Axial_L10.0mm_D6.0mm_P15.00mm_Horizontal -> Capacitor_SMD:CP_Elec_5x5.4; LCSC (none) -> C72487
- C6: footprint libraries:C_Flat_L7.2_H6.5 -> Capacitor_SMD:C_0603_1608Metric; LCSC (none) -> C14858
- C7: footprint libraries:C_Flat_L7.2_H6.5 -> Capacitor_SMD:C_0603_1608Metric; LCSC (none) -> C1588
- R1, R2, R4, R6: footprint Resistor_THT:R_Axial_DIN0207_L6.3mm_D2.5mm_P10.16mm_Horizontal -> Resistor_SMD:R_0603_1608Metric; LCSC (none) -> C22935
- R10: footprint Resistor_THT:R_Axial_DIN0207_L6.3mm_D2.5mm_P10.16mm_Horizontal -> Resistor_SMD:R_0603_1608Metric; LCSC (none) -> C25803
- R5: footprint Resistor_THT:R_Axial_DIN0207_L6.3mm_D2.5mm_P10.16mm_Horizontal -> Resistor_SMD:R_0603_1608Metric; LCSC (none) -> C25819
- R7, R8, R9: footprint Resistor_THT:R_Axial_DIN0207_L6.3mm_D2.5mm_P10.16mm_Horizontal -> Resistor_SMD:R_0603_1608Metric; LCSC (none) -> C25804
Connections:
- net +9V: now also IC2.14 (VDD)
- net GND: now also IC2.7 (VSS), R11.1, R12.1, R13.1
- net pin1: now also IC2.1 (A)
- net pin10: now also IC2.10 (K=~E)
- net pin11: now also IC2.11 (E), IC2.8 (J=~D)
- net pin12: now also IC2.12 (L=~F)
- net pin13: now also IC2.13 (F), IC2.2 (G=~A)
- net pin3: now also IC2.3 (B)
- net pin4: now also IC2.4 (H=~B)
- net pin5: now also IC2.5 (C)
- net pin6: now also IC2.6 (I=~C)
- net pin9: now also IC2.9 (D), Q1.3 (C)
- net at D1.1 (K), R3.2: now also R12.2; no longer D2.1 (K)
- net at C6.1, R7.2, R8.1: now also Q1.1 (B)
- net at C7.2, R10.1: now also Q1.2 (E)
- new net: D2.1 (K), R11.2, R13.2
Other:
- moved on the sheet: D1, D2, R3
