File: ConsolePedalDelaySMT/ConsolePedalDelaySMT.sch (KiCad schematic (older format))
At the start: 55 parts, among them J1 Conn_02x25_Counter_Clockwise, U1 TL072, U2 PT2399, U3 L78L05_TO92

Commit message: Minor changes
Parts:
- removed D1: 1N5817, Diode_SMD:D_SOD-123, symbol Diode:1N5817
- removed U3: L78L05_TO92, Package_TO_SOT_THT:TO-92_Inline, symbol Regulator_Linear:L78L05_TO92
- added R22, R24: 100K, Resistor_SMD:R_0603_1608Metric, symbol Device:R
- added R23: RLED, Resistor_THT:R_Axial_DIN0207_L6.3mm_D2.5mm_P10.16mm_Horizontal, symbol Device:R
- added U3: L78L05_SOT89, Package_TO_SOT_SMD:SOT-89-3, symbol Regulator_Linear:L78L05_SOT89
- C1, C11: footprint Capacitor_SMD:C_0805_2012Metric -> Capacitor_SMD:C_0603_1608Metric; LCSC C1729 -> C21122
- C10, C18, C19, C9: footprint Capacitor_SMD:C_0805_2012Metric -> Capacitor_SMD:C_0603_1608Metric; LCSC C49678 -> C14663
- C12: footprint Capacitor_SMD:C_0805_2012Metric -> Capacitor_SMD:C_0603_1608Metric; LCSC C1710 -> C57112
- C15: footprint Capacitor_SMD:C_0805_2012Metric -> Capacitor_SMD:C_0603_1608Metric; LCSC C53134 -> C1622
- C16: footprint Capacitor_SMD:C_0805_2012Metric -> Capacitor_SMD:C_0603_1608Metric; LCSC C52412 -> C1596
- C2: footprint Capacitor_SMD:C_0805_2012Metric -> Capacitor_SMD:C_0603_1608Metric; LCSC C14857 -> C1671
- C3: footprint Capacitor_SMD:C_0805_2012Metric -> Capacitor_SMD:C_0603_1608Metric; LCSC C1790 -> C14858
- C6: footprint Capacitor_SMD:C_0805_2012Metric -> Capacitor_SMD:C_0603_1608Metric; LCSC C1744 -> C53987
- C7, C8: footprint Capacitor_SMD:C_0805_2012Metric -> Capacitor_SMD:C_0603_1608Metric; LCSC C28260 -> C1604
- J1: footprint libraries:N64-Connector -> libraries:N64-Connector-Wide
- R21: value LED -> RLED
- U2: footprint Package_DIP:DIP-16_W7.62mm_Socket -> Package_SO:SOP-16_3.9x9.9mm_P1.27mm; LCSC (none) -> C126407
Connections:
- net +9V: now also R18.2
- net 5V: now also U3.1 (OUT)
- net GND: now also R22.1, R23.1, R24.1, U3.2 (GND)
- net at D3.1 (K), R21.2: now also R22.2; no longer D2.1 (K)
- net at C20.1, R18.1, R19.1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: now also U3.3 (IN)
- new net: D2.1 (K), R23.2, R24.2
Other:
- moved on the sheet: D2, D3, R21
