File: ConsolePedalDelaySMT/ConsolePedalDelaySMT.kicad_pcb (KiCad board)
At the start: 4 copper layers, 100 x 60 mm, 55 parts, among them J1 Conn_02x25_Counter_Clockwise, U1 TL072, U2 PT2399, U3 L78L05_TO92

Commit message: Moved around some footprints
Parts:
- C10, C11: moved to F.Cu
- Cm: renamed from C6; moved to F.Cu
- moved Cm 83.6 mm to (93.7, 98.3)
- moved R7 73.2 mm to (105.2, 108.7)
- moved C22 59.5 mm to (160.3, 105.2), turned to 270 degrees
- moved C21 57.8 mm to (119.1, 78.0), turned to 90 degrees
- moved C20 53.6 mm to (166.1, 114.6)
- moved R8 50.6 mm to (100.3, 105.2)
- moved C8 47.3 mm to (140.0, 98.8), turned to 270 degrees
- moved C9 45.7 mm to (140.0, 104.1), turned to 270 degrees
- moved R3 41.1 mm to (105.2, 101.6), turned to 180 degrees
- moved R9 37.8 mm to (105.2, 112.0), turned to 0 degrees
- moved C13 37.7 mm to (175.0, 78.0)
- moved C2 37.6 mm to (105.2, 105.2)
- moved R20 32.3 mm to (109.5, 101.6), turned to 0 degrees
- moved C18 30.0 mm to (123.7, 104.4)
- moved C5 28.6 mm to (115.1, 105.9), turned to 270 degrees
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Routing:
- net /Output: track 71.8 -> 66.0 mm
- net /pin14: track 3.30 -> 0.00 mm
- net GND: vias 6 -> 4
Other:
- board text added: "Console Pedal Delay SMT V1.0"
- board text removed: "Console Pedal Delay V1.0"

Commit message: Finalized board. Need to figure out how to export assembly instructions again.
Parts:
- moved R4 63.2 mm to (111.1, 102.0)
- moved D1 44.4 mm to (115.2, 107.1), turned to 180 degrees
- moved R11 40.5 mm to (147.4, 103.5)
- moved C20 30.9 mm to (142.5, 94.6), turned to 270 degrees
- moved C14 30.1 mm to (119.0, 76.4), turned to 90 degrees
- moved C10 30.0 mm to (140.5, 110.5), turned to 270 degrees
- moved C16 30.0 mm to (147.4, 111.1), turned to 0 degrees
- moved R17 29.9 mm to (124.5, 102.9), turned to 180 degrees
- moved R12 29.5 mm to (147.4, 105.8)
- moved C21 27.8 mm to (91.4, 76.4)
- moved R19 24.7 mm to (110.5, 96.4), turned to 270 degrees
- moved R16 24.4 mm to (147.4, 108.3), turned to 180 degrees
- moved C12 23.2 mm to (177.3, 86.7), turned to 90 degrees
- moved R10 18.9 mm to (156.5, 89.0)
- moved R6 18.8 mm to (150.4, 83.9)
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- renumbered Cm to C6
Connections:
- J1 pad 10: (no net) -> Net-(J1-Pad10)
- J1 pad 11: (no net) -> Net-(J1-Pad11)
- J1 pad 12: (no net) -> Net-(J1-Pad12)
- J1 pad 13: (no net) -> Net-(J1-Pad13)
- J1 pad 14: (no net) -> Net-(J1-Pad14)
- J1 pad 15: (no net) -> Net-(J1-Pad15)
- J1 pad 16: (no net) -> Net-(J1-Pad16)
- J1 pad 17: (no net) -> Net-(J1-Pad17)
- J1 pad 18: (no net) -> Net-(J1-Pad18)
- J1 pad 19: (no net) -> Net-(J1-Pad19)
- J1 pad 32: (no net) -> Net-(J1-Pad32)
- J1 pad 33: (no net) -> Net-(J1-Pad33)
- J1 pad 34: (no net) -> Net-(J1-Pad34)
- J1 pad 35: (no net) -> Net-(J1-Pad35)
- J1 pad 36: (no net) -> Net-(J1-Pad36)
- J1 pad 37: (no net) -> Net-(J1-Pad37)
- J1 pad 38: (no net) -> Net-(J1-Pad38)
- J1 pad 39: (no net) -> Net-(J1-Pad39)
- J1 pad 40: (no net) -> Net-(J1-Pad40)
- J1 pad 41: (no net) -> Net-(J1-Pad41)
- J1 pad 42: (no net) -> Net-(J1-Pad42)
- J1 pad 43: (no net) -> Net-(J1-Pad43)
- J1 pad 44: (no net) -> Net-(J1-Pad44)
- J1 pad 7: (no net) -> Net-(J1-Pad7)
- J1 pad 8: (no net) -> Net-(J1-Pad8)
- J1 pad 9: (no net) -> Net-(J1-Pad9)
- U2 pad 5: (no net) -> Net-(U2-Pad5)
Routing:
- net Net-(C6-Pad1): track 0.00 -> 93.7 mm, vias 0 -> 2
- net Net-(C20-Pad1): track 0.00 -> 71.8 mm
- net /5V: track 0.00 -> 69.7 mm, vias 0 -> 1
- net /pin16: track 0.00 -> 68.6 mm, vias 0 -> 2
- net Net-(C12-Pad2): track 0.00 -> 68.2 mm, vias 0 -> 2
- net /pin15: track 0.00 -> 63.1 mm, vias 0 -> 1
- net Net-(C3-Pad2): track 0.00 -> 53.5 mm
- net Net-(C13-Pad2): track 0.00 -> 51.0 mm, vias 0 -> 1
- net /LEDPower: track 54.1 -> 103.6 mm
- net /Input: track 71.6 -> 119.8 mm
- net /Output: track 66.0 -> 112.0 mm
- net Net-(D2-Pad1): track 0.00 -> 40.9 mm
- net /VREF: track 0.00 -> 38.9 mm, vias 0 -> 2
- net /pin14: track 0.00 -> 37.9 mm, vias 0 -> 1
- net /pin4: track 0.00 -> 35.3 mm, vias 0 -> 1
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- removed copper zone on In1.Cu, net GND
- removed copper zone on In2.Cu, net GND
Other:
- copper layers 4 -> 2

Commit message: Finalized assembly files and made sure everything looked ok in the jlcpcb website
Other:
- board text added: "+"
- board text added: "Thomas McDonagh consolepedals.com"
- board text removed: "Thomas McDonagh mcdonaghcorp.com"

Commit message: Minor changes
Parts:
- removed D1: 1N5817, Diode_SMD:D_SOD-123
- added R22: 100K, Resistor_SMD:R_0603_1608Metric, F.Cu at (115.2, 91.0)
- added R23: RLED, Resistor_THT:R_Axial_DIN0207_L6.3mm_D2.5mm_P10.16mm_Horizontal, F.Cu at (164.8, 91.0)
- added R24: 100K, Resistor_SMD:R_0603_1608Metric, F.Cu at (150.2, 91.0)
- C1, C10, C11, C12, C15, C16, C18, C19, C2, C3, C6, C7, C8, C9: footprint Capacitor_SMD:C_0805_2012Metric -> Capacitor_SMD:C_0603_1608Metric
- J1: footprint libraries:N64-Connector -> libraries:N64-Connector-Wide
- R21: value LED -> RLED
- U2: footprint Package_DIP:DIP-16_W7.62mm_Socket -> Package_SO:SOP-16_3.9x9.9mm_P1.27mm
- U3: value L78L05_TO92 -> L78L05_SOT89; footprint Package_TO_SOT_THT:TO-92_Inline -> Package_TO_SOT_SMD:SOT-89-3
- moved R1 64.2 mm to (160.2, 116.0)
- moved R18 59.0 mm to (174.0, 106.5)
- moved C7 49.4 mm to (142.2, 100.0), turned to 180 degrees
- moved R9 40.1 mm to (135.2, 96.3)
- moved R13 38.7 mm to (155.8, 95.0)
- moved R21 37.7 mm to (100.1, 91.0), turned to 0 degrees
- moved R8 37.6 mm to (130.2, 96.3)
- moved C6 27.9 mm to (115.2, 116.0)
- moved C11 26.8 mm to (135.2, 92.3)
- moved R10 26.4 mm to (130.2, 92.3)
- moved R7 24.9 mm to (123.2, 112.0), turned to 180 degrees
- moved C1 24.6 mm to (105.1, 116.0), turned to 0 degrees
- moved C12 21.4 mm to (159.2, 98.2), turned to 180 degrees
- moved R20 16.8 mm to (115.2, 104.0), turned to 0 degrees
- moved R15 14.6 mm to (115.2, 85.0), turned to 90 degrees
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Connections:
- D3 pad 1: Net-(D2-Pad1) -> Net-(D3-Pad1)
- J1 pad 10: Net-(J1-Pad10) -> (no net)
- J1 pad 11: Net-(J1-Pad11) -> (no net)
- J1 pad 12: Net-(J1-Pad12) -> (no net)
- J1 pad 13: Net-(J1-Pad13) -> (no net)
- J1 pad 14: Net-(J1-Pad14) -> (no net)
- J1 pad 15: Net-(J1-Pad15) -> (no net)
- J1 pad 16: Net-(J1-Pad16) -> (no net)
- J1 pad 17: Net-(J1-Pad17) -> (no net)
- J1 pad 18: Net-(J1-Pad18) -> (no net)
- J1 pad 19: Net-(J1-Pad19) -> (no net)
- J1 pad 32: Net-(J1-Pad32) -> (no net)
- J1 pad 33: Net-(J1-Pad33) -> (no net)
- J1 pad 34: Net-(J1-Pad34) -> (no net)
- J1 pad 35: Net-(J1-Pad35) -> (no net)
- J1 pad 36: Net-(J1-Pad36) -> (no net)
- J1 pad 37: Net-(J1-Pad37) -> (no net)
- J1 pad 38: Net-(J1-Pad38) -> (no net)
- J1 pad 39: Net-(J1-Pad39) -> (no net)
- J1 pad 40: Net-(J1-Pad40) -> (no net)
- J1 pad 41: Net-(J1-Pad41) -> (no net)
- J1 pad 42: Net-(J1-Pad42) -> (no net)
- J1 pad 43: Net-(J1-Pad43) -> (no net)
- J1 pad 44: Net-(J1-Pad44) -> (no net)
- J1 pad 7: Net-(J1-Pad7) -> (no net)
- J1 pad 8: Net-(J1-Pad8) -> (no net)
- J1 pad 9: Net-(J1-Pad9) -> (no net)
- R18 pad 2: Net-(D1-Pad1) -> +9V
- R21 pad 2: Net-(D2-Pad1) -> Net-(D3-Pad1)
- U2 pad 5: Net-(U2-Pad5) -> (no net)
Routing:
- net Net-(C6-Pad1): track 93.7 -> 19.3 mm, vias 2 -> 0
- net /pin16: track 68.6 -> 0.00 mm, vias 2 -> 0
- net GND: track 102.5 -> 37.5 mm, vias 20 -> 4
- net Net-(C12-Pad2): track 68.2 -> 3.96 mm, vias 2 -> 0
- net /5V: track 69.7 -> 7.92 mm, vias 1 -> 0
- net Net-(C20-Pad1): track 71.8 -> 12.1 mm
- net /pin15: track 63.1 -> 7.90 mm, vias 1 -> 0
- net Net-(C13-Pad2): track 51.0 -> 0.00 mm, vias 1 -> 0
- net /LEDPower: track 103.6 -> 53.8 mm
- net /Output: track 112.0 -> 65.7 mm
- net Net-(C3-Pad2): track 53.5 -> 8.82 mm
- net /pin14: track 37.9 -> 0.00 mm, vias 1 -> 0
- net /Input: track 119.8 -> 83.7 mm
- net /pin4: track 35.3 -> 0.00 mm, vias 1 -> 0
- net /VREF: track 38.9 -> 4.00 mm, vias 2 -> 0
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Other:
- outline, holes or cut-outs redrawn
- board text added: "Delay"
- board text added: "Delay SMT V1.1"
- board text added: "Level"
- board text added: "Repeat"
- board text removed: "+"
- board text removed: "Console Pedal Delay SMT V1.0"

Commit message: Finalized and exported new version of SMT delay cartridge PCB
Routing:
- net Net-(C20-Pad1): track 12.1 -> 123.0 mm, vias 0 -> 4
- net Net-(C13-Pad2): track 0.00 -> 68.7 mm
- net Net-(C3-Pad1): track 5.85 -> 67.1 mm, vias 0 -> 2
- net /LEDPower: track 53.8 -> 113.6 mm, vias 2 -> 6
- net Net-(C3-Pad2): track 8.82 -> 56.2 mm, vias 0 -> 2
- net /VREF: track 4.00 -> 50.3 mm, vias 0 -> 4
- net /pin4: track 0.00 -> 44.1 mm
- net /Output: track 65.7 -> 109.6 mm, vias 2 -> 4
- net /5V: track 7.92 -> 49.7 mm, vias 0 -> 2
- net Net-(R17-Pad2): track 2.50 -> 37.8 mm, vias 0 -> 1
- net Net-(C11-Pad1): track 0.00 -> 34.9 mm, vias 0 -> 1
- net Net-(C6-Pad1): track 19.3 -> 53.6 mm
- net Net-(C12-Pad2): track 3.96 -> 37.9 mm
- net +9V: track 59.7 -> 93.3 mm
- net /pin14: track 0.00 -> 28.5 mm
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